File: ATM90E36_0.sch (KiCad schematic (older format))
At the start: 20 parts, among them IC1 ATM90E36_ATM90E36, J1 GS3, J2 GS3, J3 GS3, Y1 Crystal_GND24

Commit message: Wired up current samplers
Parts:
- added C21, C22, C23, C24, C25, C26, C27, C28: 18n, Capacitors_SMD:C_0402, symbol device:C_Small
- added R11, R12, R13, R14, R15, R16, R17, R18: 1K, Resistors_SMD:R_0402, symbol device:R
- C1, C10, C2, C3, C4, C5, C6, C7, C8, C9: symbol C_Small -> device:C_Small
- IC1: symbol ATM90E36_ATM90E36 -> ATM90E36_Breakout:ATM90E36_ATM90E36
- J1, J2, J3: symbol GS3 -> conn:GS3
- R1, R2, R3, R4: symbol R -> device:R
- R5: symbol SEEED-RESISTOR-2016_SMD-RES-ARRAY-1K-4R_RA1206-8_ -> ATM90E36_Breakout:SEEED-RESISTOR-2016_SMD-RES-ARRAY-1K-4R_RA1206-8_
- Y1: symbol Crystal_GND24 -> device:Crystal_GND24
Connections:
- net labels added: IA1+, IA1-, IB1+, IB1-, IC1+, IC1-, IN1+, IN1-
- wire segments 126 -> 198

Commit message: Add part values
Parts:
- C1, C3, C5, C8: value C_Small -> 100n
- C10, C4, C9: value C_Small -> 18n
- C2, C6: value C_Small -> 10u
- R1, R2, R4: value R -> 1K
- R3: value R -> 10K
- R5: value SMD-RES-ARRAY -> SMD-RES-ARRAY_10K
Changed lines of the file:
@@
 AR Path="/5A432D2E/5A433378" Ref="R5"  Part="1"
 F 0 "R5" V 6458 2028 45  0000 L CNN
-F 1 "SMD-RES-ARRAY" V 6542 2028 45  0000 L CNN
+F 1 "SMD-RES-ARRAY_10K" V 6542 2028 45  0000 L CNN
 F 2 "Resistors_SMD:R_Array_Concave_4x0603" H 6500 1800 60  0001 C CNN
 F 3 "" H 6500 1800 60  0001 C CNN
@@
 P 3750 2400
 F 0 "C1" V 3521 2400 50  0000 C CNN
-F 1 "C_Small" V 3612 2400 50  0000 C CNN
+F 1 "100n" V 3612 2400 50  0000 C CNN
 F 2 "Capacitors_SMD:C_0402" H 3750 2400 50  0001 C CNN
 F 3 "" H 3750 2400 50  0001 C CNN
@@
 P 4400 2050
 F 0 "C5" V 4171 2050 50  0000 C CNN
-F 1 "C_Small" V 4262 2050 50  0000 C CNN
+F 1 "100n" V 4262 2050 50  0000 C CNN
 F 2 "Capacitors_SMD:C_0402" H 4400 2050 50  0001 C CNN
 F 3 "" H 4400 2050 50  0001 C CNN
@@
 P 4750 1700
 F 0 "C6" V 4521 1700 50  0000 C CNN
-F 1 "C_Small" V 4612 1700 50  0000 C CNN
+F 1 "10u" V 4612 1700 50  0000 C CNN
 F 2 "Capacitors_SMD:C_0402" H 4750 1700 50  0001 C CNN
 F 3 "" H 4750 1700 50  0001 C CNN
@@
 P 4850 1450
 F 0 "C8" V 4621 1450 50  0000 C CNN
-F 1 "C_Small" V 4712 1450 50  0000 C CNN
+F 1 "100n" V 4712 1450 50  0000 C CNN
 F 2 "Capacitors_SMD:C_0402" H 4850 1450 50  0001 C CNN
 F 3 "" H 4850 1450 50  0001 C CNN
@@
 P 3750 4250
 F 0 "C2" H 3658 4204 50  0000 R CNN
-F 1 "C_Small" H 3658 4295 50  0000 R CNN
+F 1 "10u" H 3658 4295 50  0000 R CNN
 F 2 "Capacitors_SMD:C_0603" H 3750 4250 50  0001 C CNN
 F 3 "" H 3750 4250 50  0001 C CNN
@@
 P 4000 4250
 F 0 "C3" H 3908 4204 50  0000 R CNN
-F 1 "C_Small" H 3908 4295 50  0000 R CNN
+F 1 "100n" H 3908 4295 50  0000 R CNN
 F 2 "Capacitors_SMD:C_0402" H 4000 4250 50  0001 C CNN
 F 3 "" H 4000 4250 50  0001 C CNN
@@
 P 4250 5350
 F 0 "C4" H 4158 5304 50  0000 R CNN
-F 1 "C_Small" H 4158 5395 50  0000 R CNN
+F 1 "18n" H 4158 5395 50  0000 R CNN
 F 2 "Capacitors_SMD:C_0402" H 4250 5350 50  0001 C CNN
 F 3 "" H 4250 5350 50  0001 C CNN
@@
 P 4850 5350
 F 0 "C9" H 4758 5304 50  0000 R CNN
-F 1 "C_Small" H 4758 5395 50  0000 R CNN
+F 1 "18n" H 4758 5395 50  0000 R CNN
 F 2 "Capacitors_SMD:C_0402" H 4850 5350 50  0001 C CNN
 F 3 "" H 4850 5350 50  0001 C CNN
@@
 P 5450 5350
 F 0 "C10" H 5358 5304 50  0000 R CNN
-F 1 "C_Small" H 5358 5395 50  0000 R CNN
+F 1 "18n" H 5358 5395 50  0000 R CNN
 F 2 "Capacitors_SMD:C_0402" H 5450 5350 50  0001 C CNN
 F 3 "" H 5450 5350 50  0001 C CNN
@@
 P 4050 5350
 F 0 "R1" H 4120 5396 50  0000 L CNN
-F 1 "R" H 4120 5305 50  0000 L CNN
+F 1 "1K" H 4120 5305 50  0000 L CNN
 F 2 "Resistors_SMD:R_0402" V 3980 5350 50  0001 C CNN
 F 3 "" H 4050 5350 50  0001 C CNN
@@
 P 4700 5350
 F 0 "R2" H 4770 5396 50  0000 L CNN
-F 1 "R" H 4770 5305 50  0000 L CNN
+F 1 "1K" H 4770 5305 50  0000 L CNN
 F 2 "Resistors_SMD:R_0402" V 4630 5350 50  0001 C CNN
 F 3 "" H 4700 5350 50  0001 C CNN
@@
 P 5250 5350
 F 0 "R4" H 5320 5396 50  0000 L CNN
-F 1 "R" H 5320 5305 50  0000 L CNN
+F 1 "1K" H 5320 5305 50  0000 L CNN
 F 2 "Resistors_SMD:R_0402" V 5180 5350 50  0001 C CNN
 F 3 "" H 5250 5350 50  0001 C CNN
@@
 P 5250 1450
 F 0 "R3" V 5043 1450 50  0000 C CNN
-F 1 "R" V 5134 1450 50  0000 C CNN
+F 1 "10K" V 5134 1450 50  0000 C CNN
 F 2 "Resistors_SMD:R_0402" V 5180 1450 50  0001 C CNN
 F 3 "" H 5250 1450 50  0001 C CNN

Commit message: Clean up part placement, prep for final place and route
Parts:
- C7: value C_Small -> 100n
- renumbered J1 to DMA_0, J2 to PM0_0, J3 to PM1_0
Changed lines of the file:
@@
 P 4750 1900
 F 0 "C7" V 4521 1900 50  0000 C CNN
-F 1 "C_Small" V 4612 1900 50  0000 C CNN
+F 1 "100n" V 4612 1900 50  0000 C CNN
 F 2 "Capacitors_SMD:C_0603" H 4750 1900 50  0001 C CNN
 F 3 "" H 4750 1900 50  0001 C CNN
@@
 	7050 4750 7050 4700
 $Comp
-L conn:GS3 J1
+L conn:GS3 DMA_0
 U 1 1 5A433743
 P 4350 7050
-F 0 "J1" H 4350 6725 50  0000 C CNN
+F 0 "DMA_0" H 4350 6725 50  0000 C CNN
 F 1 "GS3" H 4350 6816 50  0000 C CNN
 F 2 "Connectors:GS3" V 4438 6976 50  0001 C CNN
@@
 $EndComp
 $Comp
-L conn:GS3 J2
+L conn:GS3 PM0_0
 U 1 1 5A43374A
 P 5100 7050
-F 0 "J2" H 5100 6725 50  0000 C CNN
+F 0 "PM0_0" H 5100 6725 50  0000 C CNN
 F 1 "GS3" H 5100 6816 50  0000 C CNN
 F 2 "Connectors:GS3" V 5188 6976 50  0001 C CNN
@@
 $EndComp
 $Comp
-L conn:GS3 J3
+L conn:GS3 PM1_0
 U 1 1 5A433751
 P 5750 7050
-F 0 "J3" H 5750 6725 50  0000 C CNN
+F 0 "PM1_0" H 5750 6725 50  0000 C CNN
 F 1 "GS3" H 5750 6816 50  0000 C CNN
 F 2 "Connectors:GS3" V 5838 6976 50  0001 C CNN

Commit message: Intial work from Joslyn
Parts:
- removed C7: 100n, Capacitors_SMD:C_0603, symbol device:C_Small
- removed R5: SMD-RES-ARRAY_10K, Resistors_SMD:R_Array_Concave_4x0603, symbol ATM90E36_Breakout:SEEED-RESISTOR-2016_SMD-RES-ARRAY-1K-4R_RA1206-8_
- C3: value 100n -> 10u; footprint Capacitors_SMD:C_0402 -> Capacitors_SMD:C_0603
- C6: footprint Capacitors_SMD:C_0402 -> Capacitors_SMD:C_0603
Connections:
- wire segments 198 -> 123

Commit message: Upgrade to symbol library table format
Connections:
- wire segments 123 -> 148
Changed lines of the file:
@@
-EESchema Schematic File Version 2
-LIBS:power
+EESchema Schematic File Version 4
 LIBS:din_meter_atm90e36-cache
-EELAYER 25 0
+EELAYER 26 0
 EELAYER END
 $Descr A4 11693 8268
@@
 	4500 7150 4500 7300
 Wire Wire Line
-	4500 7300 6000 7300
+	4500 7300 5250 7300
 Wire Wire Line
 	5250 7300 5250 7150
@@
 	4500 6950 4500 6800
 Wire Wire Line
-	4500 6800 6000 6800
+	4500 6800 5250 6800
 Wire Wire Line
 	5250 6800 5250 6950
@@
 	8350 850  8600 850
 Wire Wire Line
-	8900 850  9250 850
+	8900 850  9000 850
 Wire Wire Line
 	9000 850  9000 950
@@
 	8350 1600 8600 1600
 Wire Wire Line
-	8900 1600 9250 1600
+	8900 1600 9000 1600
 Wire Wire Line
 	9000 1600 9000 1500
 Wire Wire Line
-	9000 1150 9000 1300
+	9000 1150 9000 1200
 Connection ~ 9000 1200
 Connection ~ 9000 850
@@
 	8350 2050 8600 2050
 Wire Wire Line
-	8900 2050 9250 2050
+	8900 2050 9000 2050
 Wire Wire Line
 	9000 2050 9000 2150
@@
 	8350 2800 8600 2800
 Wire Wire Line
-	8900 2800 9250 2800
+	8900 2800 9000 2800
 Wire Wire Line
 	9000 2800 9000 2700
 Wire Wire Line
-	9000 2350 9000 2500
+	9000 2350 9000 2400
 Connection ~ 9000 2400
 Connection ~ 9000 2050
@@
 	9900 850  10150 850
 Wire Wire Line
-	10450 850  10800 850
+	10450 850  10550 850
 Wire Wire Line
 	10550 850  10550 950
@@
 	9900 1600 10150 1600
 Wire Wire Line
-	10450 1600 10800 1600
+	10450 1600 10550 1600
 Wire Wire Line
 	10550 1600 10550 1500
 Wire Wire Line
-	10550 1150 10550 1300
+	10550 1150 10550 1200
 Connection ~ 10550 1200
 Connection ~ 10550 850
@@
 	9900 2050 10150 2050
 Wire Wire Line
-	10450 2050 10800 2050
+	10450 2050 10550 2050
 Wire Wire Line
 	10550 2050 10550 2150
@@
 	9900 2800 10150 2800
 Wire Wire Line
-	10450 2800 10800 2800
+	10450 2800 10550 2800
 Wire Wire Line
 	10550 2800 10550 2700
 Wire Wire Line
-	10550 2350 10550 2500
+	10550 2350 10550 2400
 Connection ~ 10550 2400
 Connection ~ 10550 2050
@@
 	3500 2150 3500 2100
 Wire Wire Line
-	3450 2100 4250 2100
-Wire Wire Line
-	3450 2400 4250 2400
+	3450 2100 3500 2100
+Wire Wire Line
+	3450 2400 3500 2400
 Wire Wire Line
 	3500 2400 3500 2350
@@
 	5600 2450 5600 2500
 Wire Wire Line
-	5400 2150 5400 2500
+	5400 2150 5400 2450
 Wire Wire Line
 	5100 2150 5150 2150
@@
 	5300 5450 5300 5500
 Wire Wire Line
-	5300 4600 5300 5250
+	5300 4600 5300 5150
 Wire Wire Line
 	5300 5150 5000 5150
@@
 	5000 5150 5000 5200
 Wire Wire Line
-	4750 5050 4750 5250
+	4750 5050 4750 5150
 Wire Wire Line
 	4750 5150 4450 5150
@@
 	4450 5150 4450 5200
 Wire Wire Line
-	4200 4950 4200 5250
+	4200 4950 4200 5150
 Wire Wire Line
 	4200 5150 3900 5150
@@
 	5250 1850 5200 1850
 Wire Wire Line
-	5450 1850 5550 1850
+	5450 1850 5500 1850
 $Comp
 L power:+3V3 #PWR030
@@
 	5500 1850 5500 2500
 Connection ~ 5500 1850
+Wire Wire Line
+	5250 7300 5900 7300
+Wire Wire Line
+	5900 7300 6000 7300
+Wire Wire Line
+	5250 6800 5900 6800
+Wire Wire Line
+	5900 6800 6000 6800
+Wire Wire Line
+	9000 1200 9000 1300
+Wire Wire Line
+	9000 850  9250 850
+Wire Wire Line
+	9000 1600 9250 1600
+Wire Wire Line
+	9000 2400 9000 2500
+Wire Wire Line
+	9000 2050 9250 2050
+Wire Wire Line
+	9000 2800 9250 2800
+Wire Wire Line
+	10550 1200 10550 1300
+Wire Wire Line
+	10550 850  10800 850
+Wire Wire Line
+	10550 1600 10800 1600
+Wire Wire Line
+	10550 2400 10550 2500
+Wire Wire Line
+	10550 2050 10800 2050
+Wire Wire Line
+	10550 2800 10800 2800
+Wire Wire Line
+	3500 2100 3900 2100
+Wire Wire Line
+	3900 2100 4250 2100
+Wire Wire Line
+	3500 2400 3900 2400
+Wire Wire Line
+	3900 2400 4250 2400
+Wire Wire Line
+	5300 5150 5300 5250
+Wire Wire Line
+	4750 5150 4750 5250
+Wire Wire Line
+	4200 5150 4200 5250
+Wire Wire Line
+	5400 2450 5400 2500
+Wire Wire Line
+	5500 1850 5550 1850
 $EndSCHEMATC

Commit message: Hard wire pads
Connections:
- wire segments 148 -> 157
Changed lines of the file:
@@
 	-1   0    0    1
 $EndComp
-Text Notes 4500 6600 0    60   ~ 0
+Text Notes 4500 6450 0    60   ~ 0
 ATM90E3X Poly Phase Metering AFE
 $Comp
@@
 	4500 6950 4500 6800
 Wire Wire Line
-	4500 6800 5250 6800
+	4500 6800 4900 6800
 Wire Wire Line
 	5250 6800 5250 6950
@@
 Connection ~ 5900 6800
 Wire Wire Line
-	5600 7050 5500 7050
-Wire Wire Line
-	4950 7050 4850 7050
-Wire Wire Line
-	4200 7050 4100 7050
+	5600 7050 5550 7050
+Wire Wire Line
+	4950 7050 4900 7050
+Wire Wire Line
+	4200 7050 4150 7050
 Wire Wire Line
 	8350 850  8600 850
@@
 	5900 7300 6000 7300
 Wire Wire Line
-	5250 6800 5900 6800
+	5250 6800 5550 6800
 Wire Wire Line
 	5900 6800 6000 6800
@@
 Wire Wire Line
 	5500 1850 5550 1850
+Wire Wire Line
+	5550 7050 5550 6800
+Connection ~ 5550 7050
+Wire Wire Line
+	5550 7050 5500 7050
+Connection ~ 5550 6800
+Wire Wire Line
+	5550 6800 5900 6800
+Wire Wire Line
+	4900 7050 4900 6800
+Connection ~ 4900 7050
+Wire Wire Line
+	4900 7050 4850 7050
+Connection ~ 4900 6800
+Wire Wire Line
+	4900 6800 5250 6800
+Wire Wire Line
+	4150 7050 4150 7300
+Wire Wire Line
+	4150 7300 4500 7300
+Connection ~ 4150 7050
+Wire Wire Line
+	4150 7050 4100 7050
+Connection ~ 4500 7300
+Text GLabel 5950 6800 1    50   Input ~ 0
++3V3
+Text GLabel 5950 7300 3    50   Input ~ 0
+GND
 $EndSCHEMATC
