File: ATM90E36_0.sch (KiCad schematic (older format))
At the start: 34 parts, among them IC1 ATM90E36_ATM90E36, Y1 Crystal_GND24

Commit message: Add some manf#
Parts:
- C3: manf# (none) -> GRM188R61A106KE69D
- C4: manf# (none) -> GRM155R71H183KA12D
- C5: manf# (none) -> GRM155R61H104KE19D
- IC1: manf# (none) -> ATM90E36A-AU-Y
- R1: manf# (none) -> RR0510P-102-D
Changed lines of the file:
@@
 F 2 "Housings_QFP:TQFP-48_7x7mm_Pitch0.5mm" H 5400 3500 60  0001 C CNN
 F 3 "" H 5400 3500 60  0001 C CNN
+F 4 "ATM90E36A-AU-Y" H 5400 3500 50  0001 C CNN "manf#"
 	1    5400 3500
 	1    0    0    -1
@@
 F 2 "Capacitors_SMD:C_0402" H 4250 2250 50  0001 C CNN
 F 3 "" H 4250 2250 50  0001 C CNN
+F 4 "GRM155R61H104KE19D" H 4250 2250 50  0001 C CNN "manf#"
 	1    4250 2250
 	-1   0    0    1
@@
 F 2 "Capacitors_SMD:C_0402" H 4200 5350 50  0001 C CNN
 F 3 "" H 4200 5350 50  0001 C CNN
+F 4 " GRM155R71H183KA12D" H 4200 5350 50  0001 C CNN "manf#"
 	1    4200 5350
 	1    0    0    1
@@
 F 2 "Resistors_SMD:R_0402" V 3830 5350 50  0001 C CNN
 F 3 "" H 3900 5350 50  0001 C CNN
+F 4 "RR0510P-102-D" H 3900 5350 50  0001 C CNN "manf#"
 	1    3900 5350
 	-1   0    0    -1
@@
 F 2 "Capacitors_SMD:C_0603" H 3900 2250 50  0001 C CNN
 F 3 "" H 3900 2250 50  0001 C CNN
+F 4 "GRM188R61A106KE69D" H 3900 2250 50  0001 C CNN "manf#"
 	1    3900 2250
 	-1   0    0    1

Commit message: New BOM output
Parts:
- C1, C8: manf# (none) -> GRM155R61H104KE19D
- C10, C21, C22, C23, C24, C25, C26, C27, C28, C9: manf# (none) -> GRM155R71H183KA12D
- C2, C6: manf# (none) -> GRM188R61A106KE69D
- C4: manf# GRM155R71H183KA12D -> GRM155R71H183KA12D
- DMA_0, PM0_0, PM1_0: DNP (none) -> (none)
- R11, R12, R13, R14, R15, R16, R17, R18, R2, R4: manf# (none) -> RR0510P-102-D
- R3: manf# (none) -> CR0402-JW-103GLFCT-ND
- Y1: manf# (none) -> ABM10-16.000MHZ-E20-T
Changed lines of the file:
@@
 F 2 "Capacitors_SMD:C_0402" H 3500 2250 50  0001 C CNN
 F 3 "" H 3500 2250 50  0001 C CNN
+F 4 "GRM155R61H104KE19D" H 3500 2250 50  0001 C CNN "manf#"
 	1    3500 2250
 	-1   0    0    1
@@
 F 2 "Capacitors_SMD:C_0402" H 5350 1850 50  0001 C CNN
 F 3 "" H 5350 1850 50  0001 C CNN
+F 4 "GRM155R61H104KE19D" H 5350 1850 50  0001 C CNN "manf#"
 	1    5350 1850
 	0    1    1    0
@@
 F 2 "Capacitors_SMD:C_0603" H 4100 4150 50  0001 C CNN
 F 3 "" H 4100 4150 50  0001 C CNN
+F 4 "GRM188R61A106KE69D" H 4100 4150 50  0001 C CNN "manf#"
 	1    4100 4150
 	1    0    0    1
@@
 F 2 "Capacitors_SMD:C_0402" H 4200 5350 50  0001 C CNN
 F 3 "" H 4200 5350 50  0001 C CNN
-F 4 " GRM155R71H183KA12D" H 4200 5350 50  0001 C CNN "manf#"
+F 4 "GRM155R71H183KA12D" H 4200 5350 50  0001 C CNN "manf#"
 	1    4200 5350
 	1    0    0    1
@@
 F 2 "Capacitors_SMD:C_0402" H 4750 5350 50  0001 C CNN
 F 3 "" H 4750 5350 50  0001 C CNN
+F 4 "GRM155R71H183KA12D" H 4750 5350 50  0001 C CNN "manf#"
 	1    4750 5350
 	1    0    0    1
@@
 F 2 "Capacitors_SMD:C_0402" H 5300 5350 50  0001 C CNN
 F 3 "" H 5300 5350 50  0001 C CNN
+F 4 "GRM155R71H183KA12D" H 5300 5350 50  0001 C CNN "manf#"
 	1    5300 5350
 	1    0    0    1
@@
 F 2 "Resistors_SMD:R_0402" V 4380 5350 50  0001 C CNN
 F 3 "" H 4450 5350 50  0001 C CNN
+F 4 "RR0510P-102-D" H 4450 5350 50  0001 C CNN "manf#"
 	1    4450 5350
 	-1   0    0    -1
@@
 F 2 "Resistors_SMD:R_0402" V 4930 5350 50  0001 C CNN
 F 3 "" H 5000 5350 50  0001 C CNN
+F 4 "RR0510P-102-D" H 5000 5350 50  0001 C CNN "manf#"
 	1    5000 5350
 	-1   0    0    -1
@@
 F 2 "Resistors_SMD:R_0402" V 5630 1850 50  0001 C CNN
 F 3 "" H 5700 1850 50  0001 C CNN
+F 4 "CR0402-JW-103GLFCT-ND" H 5700 1850 50  0001 C CNN "manf#"
 	1    5700 1850
 	0    1    1    0
@@
 F 2 "Crystals:Crystal_SMD_2520-4pin_2.5x2.0mm" H 5700 5550 50  0001 C CNN
 F 3 "" H 5700 5550 50  0001 C CNN
+F 4 "ABM10-16.000MHZ-E20-T" H 5700 5550 50  0001 C CNN "manf#"
 	1    5700 5550
 	1    0    0    -1
@@
 F 2 "Connectors:GS3" V 4438 6976 50  0001 C CNN
 F 3 "" H 4350 7050 50  0001 C CNN
+F 4 " " H 4350 7050 50  0001 C CNN "DNP"
 	1    4350 7050
 	-1   0    0    1
@@
 F 2 "Connectors:GS3" V 5188 6976 50  0001 C CNN
 F 3 "" H 5100 7050 50  0001 C CNN
+F 4 " " H 5100 7050 50  0001 C CNN "DNP"
 	1    5100 7050
 	-1   0    0    1
@@
 F 2 "Connectors:GS3" V 5838 6976 50  0001 C CNN
 F 3 "" H 5750 7050 50  0001 C CNN
+F 4 " " H 5750 7050 50  0001 C CNN "DNP"
 	1    5750 7050
 	-1   0    0    1
@@
 F 2 "Capacitors_SMD:C_0402" H 9000 1050 50  0001 C CNN
 F 3 "" H 9000 1050 50  0001 C CNN
+F 4 "GRM155R71H183KA12D" H 9000 1050 50  0001 C CNN "manf#"
 	1    9000 1050
 	1    0    0    -1
@@
 F 2 "Resistors_SMD:R_0402" V 8680 850 50  0001 C CNN
 F 3 "" H 8750 850 50  0001 C CNN
+F 4 "RR0510P-102-D" H 8750 850 50  0001 C CNN "manf#"
 	1    8750 850
 	0    1    1    0
@@
 F 2 "Capacitors_SMD:C_0402" H 9000 1400 50  0001 C CNN
 F 3 "" H 9000 1400 50  0001 C CNN
+F 4 "GRM155R71H183KA12D" H 9000 1400 50  0001 C CNN "manf#"
 	1    9000 1400
 	1    0    0    1
@@
 F 2 "Resistors_SMD:R_0402" V 8680 1600 50  0001 C CNN
 F 3 "" H 8750 1600 50  0001 C CNN
+F 4 "RR0510P-102-D" H 8750 1600 50  0001 C CNN "manf#"
 	1    8750 1600
 	0    1    -1   0
@@
 F 2 "Capacitors_SMD:C_0402" H 9000 2250 50  0001 C CNN
 F 3 "" H 9000 2250 50  0001 C CNN
+F 4 "GRM155R71H183KA12D" H 9000 2250 50  0001 C CNN "manf#"
 	1    9000 2250
 	1    0    0    -1
@@
 F 2 "Resistors_SMD:R_0402" V 8680 2050 50  0001 C CNN
 F 3 "" H 8750 2050 50  0001 C CNN
+F 4 "RR0510P-102-D" H 8750 2050 50  0001 C CNN "manf#"
 	1    8750 2050
 	0    1    1    0
@@
 F 2 "Capacitors_SMD:C_0402" H 9000 2600 50  0001 C CNN
 F 3 "" H 9000 2600 50  0001 C CNN
+F 4 "GRM155R71H183KA12D" H 9000 2600 50  0001 C CNN "manf#"
 	1    9000 2600
 	1    0    0    1
@@
 F 2 "Resistors_SMD:R_0402" V 8680 2800 50  0001 C CNN
 F 3 "" H 8750 2800 50  0001 C CNN
+F 4 "RR0510P-102-D" H 8750 2800 50  0001 C CNN "manf#"
 	1    8750 2800
 	0    1    -1   0
@@
 F 2 "Capacitors_SMD:C_0402" H 10550 1050 50  0001 C CNN
 F 3 "" H 10550 1050 50  0001 C CNN
+F 4 "GRM155R71H183KA12D" H 10550 1050 50  0001 C CNN "manf#"
 	1    10550 1050
 	1    0    0    -1
@@
 F 2 "Resistors_SMD:R_0402" V 10230 850 50  0001 C CNN
 F 3 "" H 10300 850 50  0001 C CNN
+F 4 "RR0510P-102-D" H 10300 850 50  0001 C CNN "manf#"
 	1    10300 850
 	0    1    1    0
@@
 F 2 "Capacitors_SMD:C_0402" H 10550 1400 50  0001 C CNN
 F 3 "" H 10550 1400 50  0001 C CNN
+F 4 "GRM155R71H183KA12D" H 10550 1400 50  0001 C CNN "manf#"
 	1    10550 1400
 	1    0    0    1
@@
 F 2 "Resistors_SMD:R_0402" V 10230 1600 50  0001 C CNN
 F 3 "" H 10300 1600 50  0001 C CNN
+F 4 "RR0510P-102-D" H 10300 1600 50  0001 C CNN "manf#"
 	1    10300 1600
 	0    1    -1   0
@@
 F 2 "Capacitors_SMD:C_0402" H 10550 2250 50  0001 C CNN
 F 3 "" H 10550 2250 50  0001 C CNN
+F 4 "GRM155R71H183KA12D" H 10550 2250 50  0001 C CNN "manf#"
 	1    10550 2250
 	1    0    0    -1
@@
 F 2 "Resistors_SMD:R_0402" V 10230 2050 50  0001 C CNN
 F 3 "" H 10300 2050 50  0001 C CNN
+F 4 "RR0510P-102-D" H 10300 2050 50  0001 C CNN "manf#"
 	1    10300 2050
 	0    1    1    0
@@
 F 2 "Capacitors_SMD:C_0402" H 10550 2600 50  0001 C CNN
 F 3 "" H 10550 2600 50  0001 C CNN
+F 4 "GRM155R71H183KA12D" H 10550 2600 50  0001 C CNN "manf#"
 	1    10550 2600
 	1    0    0    1
@@
 F 2 "Resistors_SMD:R_0402" V 10230 2800 50  0001 C CNN
 F 3 "" H 10300 2800 50  0001 C CNN
+F 4 "RR0510P-102-D" H 10300 2800 50  0001 C CNN "manf#"
 	1    10300 2800
 	0    1    -1   0
@@
 F 2 "Capacitors_SMD:C_0603" H 5250 2150 50  0001 C CNN
 F 3 "" H 5250 2150 50  0001 C CNN
+F 4 "GRM188R61A106KE69D" H 5250 2150 50  0001 C CNN "manf#"
 	1    5250 2150
 	0    1    1    0

Commit message: rescue symbols
Parts:
- C1, C10, C2, C21, C22, C23, C24, C25, C26, C27, C28, C3, C4, C5, C6, C8, C9: symbol device:C_Small -> din_meter_atm90e36-rescue:C_Small-device
- DMA_0, PM0_0, PM1_0: symbol conn:GS3 -> din_meter_atm90e36-rescue:GS3-conn
- R1, R11, R12, R13, R14, R15, R16, R17, R18, R2, R3, R4: symbol device:R -> din_meter_atm90e36-rescue:R-device
- Y1: symbol device:Crystal_GND24 -> din_meter_atm90e36-rescue:Crystal_GND24-device
Changed lines of the file:
@@
 $EndComp
 $Comp
-L device:C_Small C1
+L din_meter_atm90e36-rescue:C_Small-device C1
 U 1 1 5A43337F
 P 3500 2250
@@
 $EndComp
 $Comp
-L device:C_Small C5
+L din_meter_atm90e36-rescue:C_Small-device C5
 U 1 1 5A433386
 P 4250 2250
@@
 $EndComp
 $Comp
-L device:C_Small C8
+L din_meter_atm90e36-rescue:C_Small-device C8
 U 1 1 5A43339B
 P 5350 1850
@@
 $EndComp
 $Comp
-L device:C_Small C2
+L din_meter_atm90e36-rescue:C_Small-device C2
 U 1 1 5A4333A2
 P 4100 4150
@@
 $EndComp
 $Comp
-L device:C_Small C4
+L din_meter_atm90e36-rescue:C_Small-device C4
 U 1 1 5A4333B0
 P 4200 5350
@@
 $EndComp
 $Comp
-L device:C_Small C9
+L din_meter_atm90e36-rescue:C_Small-device C9
 U 1 1 5A4333B7
 P 4750 5350
@@
 $EndComp
 $Comp
-L device:C_Small C10
+L din_meter_atm90e36-rescue:C_Small-device C10
 U 1 1 5A4333BE
 P 5300 5350
@@
 $EndComp
 $Comp
-L device:R R1
+L din_meter_atm90e36-rescue:R-device R1
 U 1 1 5A4333C5
 P 3900 5350
@@
 $EndComp
 $Comp
-L device:R R2
+L din_meter_atm90e36-rescue:R-device R2
 U 1 1 5A4333CC
 P 4450 5350
@@
 $EndComp
 $Comp
-L device:R R4
+L din_meter_atm90e36-rescue:R-device R4
 U 1 1 5A4333D3
 P 5000 5350
@@
 $EndComp
 $Comp
-L device:R R3
+L din_meter_atm90e36-rescue:R-device R3
 U 1 1 5A4333DA
 P 5700 1850
@@
 $EndComp
 $Comp
-L device:Crystal_GND24 Y1
+L din_meter_atm90e36-rescue:Crystal_GND24-device Y1
 U 1 1 5A4333E1
 P 5700 5550
@@
 V3P
 $Comp
-L conn:GS3 DMA_0
+L din_meter_atm90e36-rescue:GS3-conn DMA_0
 U 1 1 5A433743
 P 4350 7050
@@
 $EndComp
 $Comp
-L conn:GS3 PM0_0
+L din_meter_atm90e36-rescue:GS3-conn PM0_0
 U 1 1 5A43374A
 P 5100 7050
@@
 $EndComp
 $Comp
-L conn:GS3 PM1_0
+L din_meter_atm90e36-rescue:GS3-conn PM1_0
 U 1 1 5A433751
 P 5750 7050
@@
 PM1_0
 $Comp
-L device:C_Small C21
+L din_meter_atm90e36-rescue:C_Small-device C21
 U 1 1 5A4C0362
 P 9000 1050
@@
 $EndComp
 $Comp
-L device:R R11
+L din_meter_atm90e36-rescue:R-device R11
 U 1 1 5A4C044E
 P 8750 850
@@
 $EndComp
 $Comp
-L device:C_Small C22
+L din_meter_atm90e36-rescue:C_Small-device C22
 U 1 1 5A4D5E43
 P 9000 1400
@@
 $EndComp
 $Comp
-L device:R R12
+L din_meter_atm90e36-rescue:R-device R12
 U 1 1 5A4D5E49
 P 8750 1600
@@
 I1N_0
 $Comp
-L device:C_Small C23
+L din_meter_atm90e36-rescue:C_Small-device C23
 U 1 1 5A520A5E
 P 9000 2250
@@
 $EndComp
 $Comp
-L device:R R13
+L din_meter_atm90e36-rescue:R-device R13
 U 1 1 5A520A64
 P 8750 2050
@@
 $EndComp
 $Comp
-L device:C_Small C24
+L din_meter_atm90e36-rescue:C_Small-device C24
 U 1 1 5A520A6D
 P 9000 2600
@@
 $EndComp
 $Comp
-L device:R R14
+L din_meter_atm90e36-rescue:R-device R14
 U 1 1 5A520A73
 P 8750 2800
@@
 I2N_0
 $Comp
-L device:C_Small C25
+L din_meter_atm90e36-rescue:C_Small-device C25
 U 1 1 5A528FE1
 P 10550 1050
@@
 $EndComp
 $Comp
-L device:R R15
+L din_meter_atm90e36-rescue:R-device R15
 U 1 1 5A528FE7
 P 10300 850
@@
 $EndComp
 $Comp
-L device:C_Small C26
+L din_meter_atm90e36-rescue:C_Small-device C26
 U 1 1 5A528FF0
 P 10550 1400
@@
 $EndComp
 $Comp
-L device:R R16
+L din_meter_atm90e36-rescue:R-device R16
 U 1 1 5A528FF6
 P 10300 1600
@@
 I3N_0
 $Comp
-L device:C_Small C27
+L din_meter_atm90e36-rescue:C_Small-device C27
 U 1 1 5A531FFB
 P 10550 2250
@@
 $EndComp
 $Comp
-L device:R R17
+L din_meter_atm90e36-rescue:R-device R17
 U 1 1 5A532001
 P 10300 2050
@@
 $EndComp
 $Comp
-L device:C_Small C28
+L din_meter_atm90e36-rescue:C_Small-device C28
 U 1 1 5A53200A
 P 10550 2600
@@
 $EndComp
 $Comp
-L device:R R18
+L din_meter_atm90e36-rescue:R-device R18
 U 1 1 5A532010
 P 10300 2800
@@
 $EndComp
 $Comp
-L device:C_Small C3
+L din_meter_atm90e36-rescue:C_Small-device C3
 U 1 1 5A4D715C
 P 3900 2250
@@
 $EndComp
 $Comp
-L device:C_Small C6
+L din_meter_atm90e36-rescue:C_Small-device C6
 U 1 1 5A433394
 P 5250 2150
