File: ATM90E36_1.sch (KiCad schematic (older format))
At the start: 20 parts, among them IC2 ATM90E36_ATM90E36, J4 GS3, J5 GS3, J6 GS3, Y2 Crystal_GND24

Commit message: Wired up current samplers
Parts:
- added C29, C30, C31, C32, C33, C34, C35, C36: 18n, Capacitors_SMD:C_0402, symbol device:C_Small
- added R19, R20, R21, R22, R23, R24, R25, R26: 1K, Resistors_SMD:R_0402, symbol device:R
- C11, C12, C13, C14, C15, C16, C17, C18, C19, C20: symbol C_Small -> device:C_Small
- IC2: symbol ATM90E36_ATM90E36 -> ATM90E36_Breakout:ATM90E36_ATM90E36
- J4, J5, J6: symbol GS3 -> conn:GS3
- R10: symbol SEEED-RESISTOR-2016_SMD-RES-ARRAY-1K-4R_RA1206-8_ -> ATM90E36_Breakout:SEEED-RESISTOR-2016_SMD-RES-ARRAY-1K-4R_RA1206-8_
- R6, R7, R8, R9: symbol R -> device:R
- Y2: symbol Crystal_GND24 -> device:Crystal_GND24
Connections:
- net labels added: I1N_1, I1P_1, I2N_1, I2P_1, I3N_1, I3P_1, IA2+, IA2-, IB2+, IB2-, IC2+, IC2-, IN2+, IN2-, IN_1, IP_1
- net labels removed: I1N, I1P, I2N, I2P, I3N, I3P, IN, IP
- wire segments 126 -> 198

Commit message: Add part values
Parts:
- C11, C13, C15, C17, C18: value C_Small -> 100n
- C12, C16: value C_Small -> 10u
- C14, C19, C20: value C_Small -> 18n
- R10: value SMD-RES-ARRAY -> SMD-RES-ARRAY_10K
- R6, R7, R9: value R -> 1K
Changed lines of the file:
@@
 AR Path="/5A433C26/5A434667" Ref="R10"  Part="1"
 F 0 "R10" V 6808 1828 45  0000 L CNN
-F 1 "SMD-RES-ARRAY" V 6892 1828 45  0000 L CNN
+F 1 "SMD-RES-ARRAY_10K" V 6892 1828 45  0000 L CNN
 F 2 "Resistors_SMD:R_Array_Concave_4x0603" H 6850 1600 60  0001 C CNN
 F 3 "" H 6850 1600 60  0001 C CNN
@@
 P 4100 2200
 F 0 "C11" V 3871 2200 50  0000 C CNN
-F 1 "C_Small" V 3962 2200 50  0000 C CNN
+F 1 "100n" V 3962 2200 50  0000 C CNN
 F 2 "Capacitors_SMD:C_0402" H 4100 2200 50  0001 C CNN
 F 3 "" H 4100 2200 50  0001 C CNN
@@
 P 4750 1850
 F 0 "C15" V 4521 1850 50  0000 C CNN
-F 1 "C_Small" V 4612 1850 50  0000 C CNN
+F 1 "100n" V 4612 1850 50  0000 C CNN
 F 2 "Capacitors_SMD:C_0402" H 4750 1850 50  0001 C CNN
 F 3 "" H 4750 1850 50  0001 C CNN
@@
 P 5100 1700
 F 0 "C17" V 4871 1700 50  0000 C CNN
-F 1 "C_Small" V 4962 1700 50  0000 C CNN
+F 1 "100n" V 4962 1700 50  0000 C CNN
 F 2 "Capacitors_SMD:C_0603" H 5100 1700 50  0001 C CNN
 F 3 "" H 5100 1700 50  0001 C CNN
@@
 P 5100 1500
 F 0 "C16" V 4871 1500 50  0000 C CNN
-F 1 "C_Small" V 4962 1500 50  0000 C CNN
+F 1 "10u" V 4962 1500 50  0000 C CNN
 F 2 "Capacitors_SMD:C_0402" H 5100 1500 50  0001 C CNN
 F 3 "" H 5100 1500 50  0001 C CNN
@@
 P 5200 1250
 F 0 "C18" V 4971 1250 50  0000 C CNN
-F 1 "C_Small" V 5062 1250 50  0000 C CNN
+F 1 "100n" V 5062 1250 50  0000 C CNN
 F 2 "Capacitors_SMD:C_0402" H 5200 1250 50  0001 C CNN
 F 3 "" H 5200 1250 50  0001 C CNN
@@
 P 4100 4050
 F 0 "C12" H 4008 4004 50  0000 R CNN
-F 1 "C_Small" H 4008 4095 50  0000 R CNN
+F 1 "10u" H 4008 4095 50  0000 R CNN
 F 2 "Capacitors_SMD:C_0603" H 4100 4050 50  0001 C CNN
 F 3 "" H 4100 4050 50  0001 C CNN
@@
 P 4350 4050
 F 0 "C13" H 4258 4004 50  0000 R CNN
-F 1 "C_Small" H 4258 4095 50  0000 R CNN
+F 1 "100n" H 4258 4095 50  0000 R CNN
 F 2 "Capacitors_SMD:C_0402" H 4350 4050 50  0001 C CNN
 F 3 "" H 4350 4050 50  0001 C CNN
@@
 P 4600 5150
 F 0 "C14" H 4508 5104 50  0000 R CNN
-F 1 "C_Small" H 4508 5195 50  0000 R CNN
+F 1 "18n" H 4508 5195 50  0000 R CNN
 F 2 "Capacitors_SMD:C_0402" H 4600 5150 50  0001 C CNN
 F 3 "" H 4600 5150 50  0001 C CNN
@@
 P 5200 5150
 F 0 "C19" H 5108 5104 50  0000 R CNN
-F 1 "C_Small" H 5108 5195 50  0000 R CNN
+F 1 "18n" H 5108 5195 50  0000 R CNN
 F 2 "Capacitors_SMD:C_0402" H 5200 5150 50  0001 C CNN
 F 3 "" H 5200 5150 50  0001 C CNN
@@
 P 5800 5150
 F 0 "C20" H 5708 5104 50  0000 R CNN
-F 1 "C_Small" H 5708 5195 50  0000 R CNN
+F 1 "18n" H 5708 5195 50  0000 R CNN
 F 2 "Capacitors_SMD:C_0402" H 5800 5150 50  0001 C CNN
 F 3 "" H 5800 5150 50  0001 C CNN
@@
 P 4400 5150
 F 0 "R6" H 4470 5196 50  0000 L CNN
-F 1 "R" H 4470 5105 50  0000 L CNN
+F 1 "1K" H 4470 5105 50  0000 L CNN
 F 2 "Resistors_SMD:R_0402" V 4330 5150 50  0001 C CNN
 F 3 "" H 4400 5150 50  0001 C CNN
@@
 P 5050 5150
 F 0 "R7" H 5120 5196 50  0000 L CNN
-F 1 "R" H 5120 5105 50  0000 L CNN
+F 1 "1K" H 5120 5105 50  0000 L CNN
 F 2 "Resistors_SMD:R_0402" V 4980 5150 50  0001 C CNN
 F 3 "" H 5050 5150 50  0001 C CNN
@@
 P 5600 5150
 F 0 "R9" H 5670 5196 50  0000 L CNN
-F 1 "R" H 5670 5105 50  0000 L CNN
+F 1 "1K" H 5670 5105 50  0000 L CNN
 F 2 "Resistors_SMD:R_0402" V 5530 5150 50  0001 C CNN
 F 3 "" H 5600 5150 50  0001 C CNN

Commit message: Clean up part placement, prep for final place and route
Parts:
- R8: value R -> 1K
- renumbered J4 to DMA_1, J5 to PM0_1, J6 to PM1_1
Connections:
- wire segments 198 -> 203
Changed lines of the file:
@@
 P 5600 1250
 F 0 "R8" V 5393 1250 50  0000 C CNN
-F 1 "R" V 5484 1250 50  0000 C CNN
+F 1 "1K" V 5484 1250 50  0000 C CNN
 F 2 "Resistors_SMD:R_0402" V 5530 1250 50  0001 C CNN
 F 3 "" H 5600 1250 50  0001 C CNN
@@
 	7400 4550 7400 4500
 $Comp
-L conn:GS3 J4
+L conn:GS3 DMA_1
 U 1 1 5A4349FF
 P 4700 6750
-F 0 "J4" H 4700 6425 50  0000 C CNN
+F 0 "DMA_1" H 4700 6425 50  0000 C CNN
 F 1 "GS3" H 4700 6516 50  0000 C CNN
 F 2 "Connectors:GS3" V 4788 6676 50  0001 C CNN
@@
 $EndComp
 $Comp
-L conn:GS3 J5
+L conn:GS3 PM0_1
 U 1 1 5A434A06
 P 5450 6750
-F 0 "J5" H 5450 6425 50  0000 C CNN
+F 0 "PM0_1" H 5450 6425 50  0000 C CNN
 F 1 "GS3" H 5450 6516 50  0000 C CNN
 F 2 "Connectors:GS3" V 5538 6676 50  0001 C CNN
@@
 $EndComp
 $Comp
-L conn:GS3 J6
+L conn:GS3 PM1_1
 U 1 1 5A434A0D
 P 6100 6750
-F 0 "J6" H 6100 6425 50  0000 C CNN
+F 0 "PM1_1" H 6100 6425 50  0000 C CNN
 F 1 "GS3" H 6100 6516 50  0000 C CNN
 F 2 "Connectors:GS3" V 6188 6676 50  0001 C CNN
@@
 	6250 6500 6350 6500
 Wire Wire Line
-	5000 1250 5000 1850
-Wire Wire Line
-	6550 1300 7000 1300
+	5000 1250 5000 1500
+Wire Wire Line
+	6550 1300 6700 1300
 $Comp
 L device:C_Small C29
@@
 Text GLabel 10750 2800 2    50   Output ~ 0
 IN_1
+Wire Wire Line
+	5000 1500 5000 1700
+Connection ~ 5000 1500
+Wire Wire Line
+	5000 1700 5000 1850
+Connection ~ 5000 1700
+Connection ~ 5200 1700
+Wire Wire Line
+	6700 1300 6800 1300
+Connection ~ 6700 1300
+Wire Wire Line
+	6800 1300 6900 1300
+Connection ~ 6800 1300
+Wire Wire Line
+	6900 1300 7000 1300
+Connection ~ 6900 1300
 $EndSCHEMATC

Commit message: Intial work from Joslyn
Parts:
- removed C13: 100n, Capacitors_SMD:C_0402, symbol device:C_Small
- removed C17: 100n, Capacitors_SMD:C_0603, symbol device:C_Small
- removed R10: SMD-RES-ARRAY_10K, Resistors_SMD:R_Array_Concave_4x0603, symbol ATM90E36_Breakout:SEEED-RESISTOR-2016_SMD-RES-ARRAY-1K-4R_RA1206-8_
- added C7: 10u, Capacitors_SMD:C_0603, symbol device:C_Small
- C16: footprint Capacitors_SMD:C_0402 -> Capacitors_SMD:C_0603
Connections:
- wire segments 203 -> 123

Commit message: Hard wire pads
Connections:
- wire segments 123 -> 157
Changed lines of the file:
@@
 	1    0    0    -1
 $EndComp
-Text Notes 4700 6750 0    60   ~ 0
+Text Notes 4700 6700 0    60   ~ 0
 ATM90E3X Poly Phase Metering AFE
 $Comp
@@
 	4850 7350 4850 7500
 Wire Wire Line
-	4850 7500 6350 7500
-Wire Wire Line
 	5600 7500 5600 7350
 Wire Wire Line
@@
 	4850 7150 4850 7000
 Wire Wire Line
-	4850 7000 6350 7000
+	4850 7000 5250 7000
 Wire Wire Line
 	5600 7000 5600 7150
@@
 Connection ~ 6250 7000
 Wire Wire Line
-	5950 7250 5850 7250
-Wire Wire Line
-	5300 7250 5200 7250
-Wire Wire Line
-	4550 7250 4450 7250
+	5950 7250 5900 7250
+Wire Wire Line
+	5300 7250 5250 7250
+Wire Wire Line
+	4550 7250 4500 7250
 $Comp
 L power:+3V3 #PWR037
@@
 	8300 850  8550 850
 Wire Wire Line
-	8850 850  9200 850
+	8850 850  8950 850
 Wire Wire Line
 	8950 850  8950 950
@@
 	8300 1600 8550 1600
 Wire Wire Line
-	8850 1600 9200 1600
+	8850 1600 8950 1600
 Wire Wire Line
 	8950 1600 8950 1500
 Wire Wire Line
-	8950 1150 8950 1300
+	8950 1150 8950 1200
 $Comp
 L power:GND #PWR039
@@
 	8300 2050 8550 2050
 Wire Wire Line
-	8850 2050 9200 2050
+	8850 2050 8950 2050
 Wire Wire Line
 	8950 2050 8950 2150
@@
 	8300 2800 8550 2800
 Wire Wire Line
-	8850 2800 9200 2800
+	8850 2800 8950 2800
 Wire Wire Line
 	8950 2800 8950 2700
 Wire Wire Line
-	8950 2350 8950 2500
+	8950 2350 8950 2400
 $Comp
 L power:GND #PWR040
@@
 	9850 850  10100 850
 Wire Wire Line
-	10400 850  10750 850
+	10400 850  10500 850
 Wire Wire Line
 	10500 850  10500 950
@@
 	9850 1600 10100 1600
 Wire Wire Line
-	10400 1600 10750 1600
+	10400 1600 10500 1600
 Wire Wire Line
 	10500 1600 10500 1500
 Wire Wire Line
-	10500 1150 10500 1300
+	10500 1150 10500 1200
 $Comp
 L power:GND #PWR041
@@
 	9850 2050 10100 2050
 Wire Wire Line
-	10400 2050 10750 2050
+	10400 2050 10500 2050
 Wire Wire Line
 	10500 2050 10500 2150
@@
 	9850 2800 10100 2800
 Wire Wire Line
-	10400 2800 10750 2800
+	10400 2800 10500 2800
 Wire Wire Line
 	10500 2800 10500 2700
 Wire Wire Line
-	10500 2350 10500 2500
+	10500 2350 10500 2400
 $Comp
 L power:GND #PWR042
@@
 	4500 1800 4500 1850
 Wire Wire Line
-	3800 1800 4500 1800
+	3800 1800 3850 1800
 Wire Wire Line
 	3850 1800 3850 1850
@@
 	4500 2100 4500 2050
 Wire Wire Line
-	3800 2100 4500 2100
+	3800 2100 3850 2100
 Wire Wire Line
 	3850 2100 3850 2050
@@
 	5600 1600 5550 1600
 Wire Wire Line
-	5800 1600 5900 1600
+	5800 1600 5850 1600
 $Comp
 L power:+3V3 #PWR049
@@
 	5700 1950 5750 1950
 Wire Wire Line
-	5750 1950 5750 2300
+	5750 1950 5750 2250
 Wire Wire Line
 	5750 2250 5650 2250
@@
 	5650 5300 5650 5250
 Wire Wire Line
-	5650 4400 5650 5050
+	5650 4400 5650 4950
 Wire Wire Line
 	5650 4950 5350 4950
@@
 	5350 4950 5350 5000
 Wire Wire Line
-	5100 4850 5100 5050
+	5100 4850 5100 4950
 Wire Wire Line
 	5100 4950 4800 4950
@@
 	4800 4950 4800 5000
 Wire Wire Line
-	4550 4750 4550 5050
+	4550 4750 4550 4950
 Wire Wire Line
 	4550 4950 4250 4950
@@
 Wire Wire Line
 	6250 4850 5950 4850
+Wire Wire Line
+	5600 7500 6250 7500
+Wire Wire Line
+	6250 7500 6350 7500
+Wire Wire Line
+	5600 7000 5900 7000
+Wire Wire Line
+	6250 7000 6350 7000
+Wire Wire Line
+	8950 1200 8950 1300
+Wire Wire Line
+	8950 850  9200 850
+Wire Wire Line
+	8950 1600 9200 1600
+Wire Wire Line
+	8950 2400 8950 2500
+Wire Wire Line
+	8950 2050 9200 2050
+Wire Wire Line
+	8950 2800 9200 2800
+Wire Wire Line
+	10500 1200 10500 1300
+Wire Wire Line
+	10500 850  10750 850
+Wire Wire Line
+	10500 1600 10750 1600
+Wire Wire Line
+	10500 2400 10500 2500
+Wire Wire Line
+	10500 2050 10750 2050
+Wire Wire Line
+	10500 2800 10750 2800
+Wire Wire Line
+	4200 2100 4500 2100
+Wire Wire Line
+	4200 1800 4500 1800
+Wire Wire Line
+	3850 2100 4200 2100
+Wire Wire Line
+	3850 1800 4200 1800
+Wire Wire Line
+	5750 2250 5750 2300
+Wire Wire Line
+	5850 1600 5900 1600
+Wire Wire Line
+	5650 4950 5650 5050
+Wire Wire Line
+	5100 4950 5100 5050
+Wire Wire Line
+	4550 4950 4550 5050
+Wire Wire Line
+	4500 7250 4500 7500
+Wire Wire Line
+	4500 7500 4850 7500
+Connection ~ 4500 7250
+Wire Wire Line
+	4500 7250 4450 7250
+Connection ~ 4850 7500
+Wire Wire Line
+	4850 7500 5600 7500
+Wire Wire Line
+	5250 7250 5250 7000
+Connection ~ 5250 7250
+Wire Wire Line
+	5250 7250 5200 7250
+Connection ~ 5250 7000
+Wire Wire Line
+	5250 7000 5600 7000
+Wire Wire Line
+	5900 7250 5900 7000
+Connection ~ 5900 7250
+Wire Wire Line
+	5900 7250 5850 7250
+Connection ~ 5900 7000
+Wire Wire Line
+	5900 7000 6250 7000
+Text GLabel 6300 7000 1    50   Input ~ 0
++3V3
+Text GLabel 6300 7500 3    50   Input ~ 0
+GND
 $EndSCHEMATC

Commit message: Fixed 1k reset resistor to 10k
Parts:
- R8: value 1K -> 10K; manf# (none) -> (none)
Changed lines of the file:
@@
 P 6050 1600
 F 0 "R8" V 5843 1600 50  0000 C CNN
-F 1 "1K" V 5934 1600 50  0000 C CNN
+F 1 "10K" V 5934 1600 50  0000 C CNN
 F 2 "Resistors_SMD:R_0402" V 5980 1600 50  0001 C CNN
 F 3 "" H 6050 1600 50  0001 C CNN
+F 4 " " H 6050 1600 50  0001 C CNN "manf#"
 	1    6050 1600
 	0    1    1    0
