File: ATM90E36_1.sch (KiCad schematic (older format))
At the start: 34 parts, among them IC2 ATM90E36_ATM90E36, Y2 Crystal_GND24

Commit message: New BOM output
Parts:
- C11, C15, C18: manf# (none) -> GRM155R61H104KE19D
- C12, C16, C7: manf# (none) -> GRM188R61A106KE69D
- C14, C19, C20, C29, C30, C31, C32, C33, C34, C35, C36: manf# (none) -> GRM155R71H183KA12D
- DMA_1, PM0_1, PM1_1: DNP (none) -> (none)
- IC2: manf# (none) -> ATM90E36A-AU-Y
- R19, R20, R21, R22, R23, R24, R25, R26, R6, R7, R9: manf# (none) -> RR0510P-102-D
- R8: manf# (none) -> CR0402-JW-103GLFCT-ND
- Y2: manf# (none) -> ABM10-16.000MHZ-E20-T
Changed lines of the file:
@@
 F 2 "Housings_QFP:TQFP-48_7x7mm_Pitch0.5mm" H 5750 3300 60  0001 C CNN
 F 3 "" H 5750 3300 60  0001 C CNN
+F 4 "ATM90E36A-AU-Y" H 5750 3300 50  0001 C CNN "manf#"
 	1    5750 3300
 	1    0    0    -1
@@
 F 2 "Capacitors_SMD:C_0402" H 3850 1950 50  0001 C CNN
 F 3 "" H 3850 1950 50  0001 C CNN
+F 4 "GRM155R61H104KE19D" H 3850 1950 50  0001 C CNN "manf#"
 	1    3850 1950
 	-1   0    0    1
@@
 F 2 "Capacitors_SMD:C_0402" H 4500 1950 50  0001 C CNN
 F 3 "" H 4500 1950 50  0001 C CNN
+F 4 "GRM155R61H104KE19D" H 4500 1950 50  0001 C CNN "manf#"
 	1    4500 1950
 	-1   0    0    1
@@
 F 2 "Capacitors_SMD:C_0603" H 5600 1950 50  0001 C CNN
 F 3 "" H 5600 1950 50  0001 C CNN
+F 4 "GRM188R61A106KE69D" H 5600 1950 50  0001 C CNN "manf#"
 	1    5600 1950
 	0    1    1    0
@@
 F 2 "Capacitors_SMD:C_0402" H 5700 1600 50  0001 C CNN
 F 3 "" H 5700 1600 50  0001 C CNN
+F 4 "GRM155R61H104KE19D" H 5700 1600 50  0001 C CNN "manf#"
 	1    5700 1600
 	0    1    1    0
@@
 F 2 "Capacitors_SMD:C_0603" H 4450 3950 50  0001 C CNN
 F 3 "" H 4450 3950 50  0001 C CNN
+F 4 "GRM188R61A106KE69D" H 4450 3950 50  0001 C CNN "manf#"
 	1    4450 3950
 	1    0    0    1
@@
 F 2 "Capacitors_SMD:C_0402" H 4550 5150 50  0001 C CNN
 F 3 "" H 4550 5150 50  0001 C CNN
+F 4 "GRM155R71H183KA12D" H 4550 5150 50  0001 C CNN "manf#"
 	1    4550 5150
 	1    0    0    1
@@
 F 2 "Capacitors_SMD:C_0402" H 5100 5150 50  0001 C CNN
 F 3 "" H 5100 5150 50  0001 C CNN
+F 4 "GRM155R71H183KA12D" H 5100 5150 50  0001 C CNN "manf#"
 	1    5100 5150
 	1    0    0    1
@@
 F 2 "Capacitors_SMD:C_0402" H 5650 5150 50  0001 C CNN
 F 3 "" H 5650 5150 50  0001 C CNN
+F 4 "GRM155R71H183KA12D" H 5650 5150 50  0001 C CNN "manf#"
 	1    5650 5150
 	1    0    0    1
@@
 F 2 "Resistors_SMD:R_0402" V 4180 5150 50  0001 C CNN
 F 3 "" H 4250 5150 50  0001 C CNN
+F 4 "RR0510P-102-D" H 4250 5150 50  0001 C CNN "manf#"
 	1    4250 5150
 	-1   0    0    -1
@@
 F 2 "Resistors_SMD:R_0402" V 4730 5150 50  0001 C CNN
 F 3 "" H 4800 5150 50  0001 C CNN
+F 4 "RR0510P-102-D" H 4800 5150 50  0001 C CNN "manf#"
 	1    4800 5150
 	-1   0    0    -1
@@
 F 2 "Resistors_SMD:R_0402" V 5280 5150 50  0001 C CNN
 F 3 "" H 5350 5150 50  0001 C CNN
+F 4 "RR0510P-102-D" H 5350 5150 50  0001 C CNN "manf#"
 	1    5350 5150
 	-1   0    0    -1
@@
 F 2 "Resistors_SMD:R_0402" V 5980 1600 50  0001 C CNN
 F 3 "" H 6050 1600 50  0001 C CNN
-F 4 " " H 6050 1600 50  0001 C CNN "manf#"
+F 4 "CR0402-JW-103GLFCT-ND" H 6050 1600 50  0001 C CNN "manf#"
 	1    6050 1600
 	0    1    1    0
@@
 F 2 "Crystals:Crystal_SMD_2520-4pin_2.5x2.0mm" H 6050 5350 50  0001 C CNN
 F 3 "" H 6050 5350 50  0001 C CNN
+F 4 "ABM10-16.000MHZ-E20-T" H 6050 5350 50  0001 C CNN "manf#"
 	1    6050 5350
 	1    0    0    -1
@@
 F 2 "Connectors:GS3" V 4788 7176 50  0001 C CNN
 F 3 "" H 4700 7250 50  0001 C CNN
+F 4 " " H 4700 7250 50  0001 C CNN "DNP"
 	1    4700 7250
 	-1   0    0    1
@@
 F 2 "Connectors:GS3" V 5538 7176 50  0001 C CNN
 F 3 "" H 5450 7250 50  0001 C CNN
+F 4 " " H 5450 7250 50  0001 C CNN "DNP"
 	1    5450 7250
 	-1   0    0    1
@@
 F 2 "Connectors:GS3" V 6188 7176 50  0001 C CNN
 F 3 "" H 6100 7250 50  0001 C CNN
+F 4 " " H 6100 7250 50  0001 C CNN "DNP"
 	1    6100 7250
 	-1   0    0    1
@@
 F 2 "Capacitors_SMD:C_0402" H 8950 1050 50  0001 C CNN
 F 3 "" H 8950 1050 50  0001 C CNN
+F 4 "GRM155R71H183KA12D" H 8950 1050 50  0001 C CNN "manf#"
 	1    8950 1050
 	1    0    0    -1
@@
 F 2 "Resistors_SMD:R_0402" V 8630 850 50  0001 C CNN
 F 3 "" H 8700 850 50  0001 C CNN
+F 4 "RR0510P-102-D" H 8700 850 50  0001 C CNN "manf#"
 	1    8700 850
 	0    1    1    0
@@
 F 2 "Capacitors_SMD:C_0402" H 8950 1400 50  0001 C CNN
 F 3 "" H 8950 1400 50  0001 C CNN
+F 4 "GRM155R71H183KA12D" H 8950 1400 50  0001 C CNN "manf#"
 	1    8950 1400
 	1    0    0    1
@@
 F 2 "Resistors_SMD:R_0402" V 8630 1600 50  0001 C CNN
 F 3 "" H 8700 1600 50  0001 C CNN
+F 4 "RR0510P-102-D" H 8700 1600 50  0001 C CNN "manf#"
 	1    8700 1600
 	0    1    -1   0
@@
 F 2 "Capacitors_SMD:C_0402" H 8950 2250 50  0001 C CNN
 F 3 "" H 8950 2250 50  0001 C CNN
+F 4 "GRM155R71H183KA12D" H 8950 2250 50  0001 C CNN "manf#"
 	1    8950 2250
 	1    0    0    -1
@@
 F 2 "Resistors_SMD:R_0402" V 8630 2050 50  0001 C CNN
 F 3 "" H 8700 2050 50  0001 C CNN
+F 4 "RR0510P-102-D" H 8700 2050 50  0001 C CNN "manf#"
 	1    8700 2050
 	0    1    1    0
@@
 F 2 "Capacitors_SMD:C_0402" H 8950 2600 50  0001 C CNN
 F 3 "" H 8950 2600 50  0001 C CNN
+F 4 "GRM155R71H183KA12D" H 8950 2600 50  0001 C CNN "manf#"
 	1    8950 2600
 	1    0    0    1
@@
 F 2 "Resistors_SMD:R_0402" V 8630 2800 50  0001 C CNN
 F 3 "" H 8700 2800 50  0001 C CNN
+F 4 "RR0510P-102-D" H 8700 2800 50  0001 C CNN "manf#"
 	1    8700 2800
 	0    1    -1   0
@@
 F 2 "Capacitors_SMD:C_0402" H 10500 1050 50  0001 C CNN
 F 3 "" H 10500 1050 50  0001 C CNN
+F 4 "GRM155R71H183KA12D" H 10500 1050 50  0001 C CNN "manf#"
 	1    10500 1050
 	1    0    0    -1
@@
 F 2 "Resistors_SMD:R_0402" V 10180 850 50  0001 C CNN
 F 3 "" H 10250 850 50  0001 C CNN
+F 4 "RR0510P-102-D" H 10250 850 50  0001 C CNN "manf#"
 	1    10250 850
 	0    1    1    0
@@
 F 2 "Capacitors_SMD:C_0402" H 10500 1400 50  0001 C CNN
 F 3 "" H 10500 1400 50  0001 C CNN
+F 4 "GRM155R71H183KA12D" H 10500 1400 50  0001 C CNN "manf#"
 	1    10500 1400
 	1    0    0    1
@@
 F 2 "Resistors_SMD:R_0402" V 10180 1600 50  0001 C CNN
 F 3 "" H 10250 1600 50  0001 C CNN
+F 4 "RR0510P-102-D" H 10250 1600 50  0001 C CNN "manf#"
 	1    10250 1600
 	0    1    -1   0
@@
 F 2 "Capacitors_SMD:C_0402" H 10500 2250 50  0001 C CNN
 F 3 "" H 10500 2250 50  0001 C CNN
+F 4 "GRM155R71H183KA12D" H 10500 2250 50  0001 C CNN "manf#"
 	1    10500 2250
 	1    0    0    -1
@@
 F 2 "Resistors_SMD:R_0402" V 10180 2050 50  0001 C CNN
 F 3 "" H 10250 2050 50  0001 C CNN
+F 4 "RR0510P-102-D" H 10250 2050 50  0001 C CNN "manf#"
 	1    10250 2050
 	0    1    1    0
@@
 F 2 "Capacitors_SMD:C_0402" H 10500 2600 50  0001 C CNN
 F 3 "" H 10500 2600 50  0001 C CNN
+F 4 "GRM155R71H183KA12D" H 10500 2600 50  0001 C CNN "manf#"
 	1    10500 2600
 	1    0    0    1
@@
 F 2 "Resistors_SMD:R_0402" V 10180 2800 50  0001 C CNN
 F 3 "" H 10250 2800 50  0001 C CNN
+F 4 "RR0510P-102-D" H 10250 2800 50  0001 C CNN "manf#"
 	1    10250 2800
 	0    1    -1   0
@@
 F 2 "Capacitors_SMD:C_0603" H 4200 1950 50  0001 C CNN
 F 3 "" H 4200 1950 50  0001 C CNN
+F 4 "GRM188R61A106KE69D" H 4200 1950 50  0001 C CNN "manf#"
 	1    4200 1950
 	-1   0    0    1

Commit message: rescue symbols
Parts:
- C11, C12, C14, C15, C16, C18, C19, C20, C29, C30, C31, C32, C33, C34, C35, C36, C7: symbol device:C_Small -> din_meter_atm90e36-rescue:C_Small-device
- DMA_1, PM0_1, PM1_1: symbol conn:GS3 -> din_meter_atm90e36-rescue:GS3-conn
- R19, R20, R21, R22, R23, R24, R25, R26, R6, R7, R8, R9: symbol device:R -> din_meter_atm90e36-rescue:R-device
- Y2: symbol device:Crystal_GND24 -> din_meter_atm90e36-rescue:Crystal_GND24-device
Changed lines of the file:
@@
 ATM90E3X Poly Phase Metering AFE
 $Comp
-L device:C_Small C11
+L din_meter_atm90e36-rescue:C_Small-device C11
 U 1 1 5A43466E
 P 3850 1950
@@
 $EndComp
 $Comp
-L device:C_Small C15
+L din_meter_atm90e36-rescue:C_Small-device C15
 U 1 1 5A434675
 P 4500 1950
@@
 $EndComp
 $Comp
-L device:C_Small C16
+L din_meter_atm90e36-rescue:C_Small-device C16
 U 1 1 5A434683
 P 5600 1950
@@
 $EndComp
 $Comp
-L device:C_Small C18
+L din_meter_atm90e36-rescue:C_Small-device C18
 U 1 1 5A43468A
 P 5700 1600
@@
 $EndComp
 $Comp
-L device:C_Small C12
+L din_meter_atm90e36-rescue:C_Small-device C12
 U 1 1 5A434691
 P 4450 3950
@@
 $EndComp
 $Comp
-L device:C_Small C14
+L din_meter_atm90e36-rescue:C_Small-device C14
 U 1 1 5A43469F
 P 4550 5150
@@
 $EndComp
 $Comp
-L device:C_Small C19
+L din_meter_atm90e36-rescue:C_Small-device C19
 U 1 1 5A4346A6
 P 5100 5150
@@
 $EndComp
 $Comp
-L device:C_Small C20
+L din_meter_atm90e36-rescue:C_Small-device C20
 U 1 1 5A4346AD
 P 5650 5150
@@
 $EndComp
 $Comp
-L device:R R6
+L din_meter_atm90e36-rescue:R-device R6
 U 1 1 5A4346B4
 P 4250 5150
@@
 $EndComp
 $Comp
-L device:R R7
+L din_meter_atm90e36-rescue:R-device R7
 U 1 1 5A4346BB
 P 4800 5150
@@
 $EndComp
 $Comp
-L device:R R9
+L din_meter_atm90e36-rescue:R-device R9
 U 1 1 5A4346C2
 P 5350 5150
@@
 $EndComp
 $Comp
-L device:R R8
+L din_meter_atm90e36-rescue:R-device R8
 U 1 1 5A4346C9
 P 6050 1600
@@
 $EndComp
 $Comp
-L device:Crystal_GND24 Y2
+L din_meter_atm90e36-rescue:Crystal_GND24-device Y2
 U 1 1 5A4346D0
 P 6050 5350
@@
 V3P
 $Comp
-L conn:GS3 DMA_1
+L din_meter_atm90e36-rescue:GS3-conn DMA_1
 U 1 1 5A4349FF
 P 4700 7250
@@
 $EndComp
 $Comp
-L conn:GS3 PM0_1
+L din_meter_atm90e36-rescue:GS3-conn PM0_1
 U 1 1 5A434A06
 P 5450 7250
@@
 $EndComp
 $Comp
-L conn:GS3 PM1_1
+L din_meter_atm90e36-rescue:GS3-conn PM1_1
 U 1 1 5A434A0D
 P 6100 7250
@@
 PM1_1
 $Comp
-L device:C_Small C29
+L din_meter_atm90e36-rescue:C_Small-device C29
 U 1 1 5A53D22E
 P 8950 1050
@@
 $EndComp
 $Comp
-L device:R R19
+L din_meter_atm90e36-rescue:R-device R19
 U 1 1 5A53D235
 P 8700 850
@@
 	8950 850  8950 950
 $Comp
-L device:C_Small C30
+L din_meter_atm90e36-rescue:C_Small-device C30
 U 1 1 5A53D23F
 P 8950 1400
@@
 $EndComp
 $Comp
-L device:R R20
+L din_meter_atm90e36-rescue:R-device R20
 U 1 1 5A53D246
 P 8700 1600
@@
 I1N_1
 $Comp
-L device:C_Small C31
+L din_meter_atm90e36-rescue:C_Small-device C31
 U 1 1 5A53D261
 P 8950 2250
@@
 $EndComp
 $Comp
-L device:R R21
+L din_meter_atm90e36-rescue:R-device R21
 U 1 1 5A53D268
 P 8700 2050
@@
 	8950 2050 8950 2150
 $Comp
-L device:C_Small C32
+L din_meter_atm90e36-rescue:C_Small-device C32
 U 1 1 5A53D272
 P 8950 2600
@@
 $EndComp
 $Comp
-L device:R R22
+L din_meter_atm90e36-rescue:R-device R22
 U 1 1 5A53D279
 P 8700 2800
@@
 I2N_1
 $Comp
-L device:C_Small C33
+L din_meter_atm90e36-rescue:C_Small-device C33
 U 1 1 5A53D294
 P 10500 1050
@@
 $EndComp
 $Comp
-L device:R R23
+L din_meter_atm90e36-rescue:R-device R23
 U 1 1 5A53D29B
 P 10250 850
@@
 	10500 850  10500 950
 $Comp
-L device:C_Small C34
+L din_meter_atm90e36-rescue:C_Small-device C34
 U 1 1 5A53D2A5
 P 10500 1400
@@
 $EndComp
 $Comp
-L device:R R24
+L din_meter_atm90e36-rescue:R-device R24
 U 1 1 5A53D2AC
 P 10250 1600
@@
 I3N_1
 $Comp
-L device:C_Small C35
+L din_meter_atm90e36-rescue:C_Small-device C35
 U 1 1 5A53D2C7
 P 10500 2250
@@
 $EndComp
 $Comp
-L device:R R25
+L din_meter_atm90e36-rescue:R-device R25
 U 1 1 5A53D2CE
 P 10250 2050
@@
 	10500 2050 10500 2150
 $Comp
-L device:C_Small C36
+L din_meter_atm90e36-rescue:C_Small-device C36
 U 1 1 5A53D2D8
 P 10500 2600
@@
 $EndComp
 $Comp
-L device:R R26
+L din_meter_atm90e36-rescue:R-device R26
 U 1 1 5A53D2DF
 P 10250 2800
@@
 	6250 2250 6250 2300
 $Comp
-L device:C_Small C7
+L din_meter_atm90e36-rescue:C_Small-device C7
 U 1 1 5A4E40A6
 P 4200 1950
