File: din_meter_atm90e36.sch (KiCad schematic (older format))
At the start: 54 parts, among them IC1 ATM90E36_ATM90E36, IC2 ATM90E36_ATM90E36, J1 GS3, J2 GS3, J3 GS3, J4 GS3, J5 GS3, J6 GS3, Y1 Crystal_GND24, Y2 Crystal_GND24

Commit message: Make passives smaller
Parts:
- C1, C10, C11, C13, C14, C15, C16, C18, C19, C20, C3, C4, C5, C6, C8, C9: footprint Capacitors_SMD:C_0603 -> Capacitors_SMD:C_0402
- C12, C17, C2, C7: footprint Capacitors_SMD:C_0805 -> Capacitors_SMD:C_0603
- R1, R10, R11, R2, R4, R5, R8, R9: footprint Resistors_SMD:R_0603 -> Resistors_SMD:R_0402
Changed lines of the file:
@@
 $Descr A4 11693 8268
 encoding utf-8
-Sheet 1 1
+Sheet 1 2
 Title ""
 Date ""
@@
 F 0 "C1" V 1021 1900 50  0000 C CNN
 F 1 "C_Small" V 1112 1900 50  0000 C CNN
-F 2 "Capacitors_SMD:C_0603" H 1250 1900 50  0001 C CNN
+F 2 "Capacitors_SMD:C_0402" H 1250 1900 50  0001 C CNN
 F 3 "" H 1250 1900 50  0001 C CNN
 	1    1250 1900
@@
 F 0 "C5" V 1671 1550 50  0000 C CNN
 F 1 "C_Small" V 1762 1550 50  0000 C CNN
-F 2 "Capacitors_SMD:C_0603" H 1900 1550 50  0001 C CNN
+F 2 "Capacitors_SMD:C_0402" H 1900 1550 50  0001 C CNN
 F 3 "" H 1900 1550 50  0001 C CNN
 	1    1900 1550
@@
 F 0 "C7" V 2021 1400 50  0000 C CNN
 F 1 "C_Small" V 2112 1400 50  0000 C CNN
-F 2 "Capacitors_SMD:C_0805" H 2250 1400 50  0001 C CNN
+F 2 "Capacitors_SMD:C_0603" H 2250 1400 50  0001 C CNN
 F 3 "" H 2250 1400 50  0001 C CNN
 	1    2250 1400
@@
 F 0 "C6" V 2021 1200 50  0000 C CNN
 F 1 "C_Small" V 2112 1200 50  0000 C CNN
-F 2 "Capacitors_SMD:C_0603" H 2250 1200 50  0001 C CNN
+F 2 "Capacitors_SMD:C_0402" H 2250 1200 50  0001 C CNN
 F 3 "" H 2250 1200 50  0001 C CNN
 	1    2250 1200
@@
 F 0 "C8" V 2121 950 50  0000 C CNN
 F 1 "C_Small" V 2212 950 50  0000 C CNN
-F 2 "Capacitors_SMD:C_0603" H 2350 950 50  0001 C CNN
+F 2 "Capacitors_SMD:C_0402" H 2350 950 50  0001 C CNN
 F 3 "" H 2350 950 50  0001 C CNN
 	1    2350 950
@@
 F 0 "C2" H 1158 3704 50  0000 R CNN
 F 1 "C_Small" H 1158 3795 50  0000 R CNN
-F 2 "Capacitors_SMD:C_0805" H 1250 3750 50  0001 C CNN
+F 2 "Capacitors_SMD:C_0603" H 1250 3750 50  0001 C CNN
 F 3 "" H 1250 3750 50  0001 C CNN
 	1    1250 3750
@@
 F 0 "C3" H 1408 3704 50  0000 R CNN
 F 1 "C_Small" H 1408 3795 50  0000 R CNN
-F 2 "Capacitors_SMD:C_0603" H 1500 3750 50  0001 C CNN
+F 2 "Capacitors_SMD:C_0402" H 1500 3750 50  0001 C CNN
 F 3 "" H 1500 3750 50  0001 C CNN
 	1    1500 3750
@@
 F 0 "C4" H 1658 4804 50  0000 R CNN
 F 1 "C_Small" H 1658 4895 50  0000 R CNN
-F 2 "Capacitors_SMD:C_0603" H 1750 4850 50  0001 C CNN
+F 2 "Capacitors_SMD:C_0402" H 1750 4850 50  0001 C CNN
 F 3 "" H 1750 4850 50  0001 C CNN
 	1    1750 4850
@@
 F 0 "C9" H 2258 4804 50  0000 R CNN
 F 1 "C_Small" H 2258 4895 50  0000 R CNN
-F 2 "Capacitors_SMD:C_0603" H 2350 4850 50  0001 C CNN
+F 2 "Capacitors_SMD:C_0402" H 2350 4850 50  0001 C CNN
 F 3 "" H 2350 4850 50  0001 C CNN
 	1    2350 4850
@@
 F 0 "C10" H 2858 4804 50  0000 R CNN
 F 1 "C_Small" H 2858 4895 50  0000 R CNN
-F 2 "Capacitors_SMD:C_0603" H 2950 4850 50  0001 C CNN
+F 2 "Capacitors_SMD:C_0402" H 2950 4850 50  0001 C CNN
 F 3 "" H 2950 4850 50  0001 C CNN
 	1    2950 4850
@@
 F 0 "R1" H 1620 4896 50  0000 L CNN
 F 1 "R" H 1620 4805 50  0000 L CNN
-F 2 "Resistors_SMD:R_0603" V 1480 4850 50  0001 C CNN
+F 2 "Resistors_SMD:R_0402" V 1480 4850 50  0001 C CNN
 F 3 "" H 1550 4850 50  0001 C CNN
 	1    1550 4850
@@
 F 0 "R2" H 2270 4896 50  0000 L CNN
 F 1 "R" H 2270 4805 50  0000 L CNN
-F 2 "Resistors_SMD:R_0603" V 2130 4850 50  0001 C CNN
+F 2 "Resistors_SMD:R_0402" V 2130 4850 50  0001 C CNN
 F 3 "" H 2200 4850 50  0001 C CNN
 	1    2200 4850
@@
 F 0 "R5" H 2820 4896 50  0000 L CNN
 F 1 "R" H 2820 4805 50  0000 L CNN
-F 2 "Resistors_SMD:R_0603" V 2680 4850 50  0001 C CNN
+F 2 "Resistors_SMD:R_0402" V 2680 4850 50  0001 C CNN
 F 3 "" H 2750 4850 50  0001 C CNN
 	1    2750 4850
@@
 F 0 "R4" V 2543 950 50  0000 C CNN
 F 1 "R" V 2634 950 50  0000 C CNN
-F 2 "Resistors_SMD:R_0603" V 2680 950 50  0001 C CNN
+F 2 "Resistors_SMD:R_0402" V 2680 950 50  0001 C CNN
 F 3 "" H 2750 950 50  0001 C CNN
 	1    2750 950
@@
 F 0 "C11" V 6171 2000 50  0000 C CNN
 F 1 "C_Small" V 6262 2000 50  0000 C CNN
-F 2 "Capacitors_SMD:C_0603" H 6400 2000 50  0001 C CNN
+F 2 "Capacitors_SMD:C_0402" H 6400 2000 50  0001 C CNN
 F 3 "" H 6400 2000 50  0001 C CNN
 	1    6400 2000
@@
 F 0 "C15" V 6821 1650 50  0000 C CNN
 F 1 "C_Small" V 6912 1650 50  0000 C CNN
-F 2 "Capacitors_SMD:C_0603" H 7050 1650 50  0001 C CNN
+F 2 "Capacitors_SMD:C_0402" H 7050 1650 50  0001 C CNN
 F 3 "" H 7050 1650 50  0001 C CNN
 	1    7050 1650
@@
 F 0 "C17" V 7171 1500 50  0000 C CNN
 F 1 "C_Small" V 7262 1500 50  0000 C CNN
-F 2 "Capacitors_SMD:C_0805" H 7400 1500 50  0001 C CNN
+F 2 "Capacitors_SMD:C_0603" H 7400 1500 50  0001 C CNN
 F 3 "" H 7400 1500 50  0001 C CNN
 	1    7400 1500
@@
 F 0 "C16" V 7171 1300 50  0000 C CNN
 F 1 "C_Small" V 7262 1300 50  0000 C CNN
-F 2 "Capacitors_SMD:C_0603" H 7400 1300 50  0001 C CNN
+F 2 "Capacitors_SMD:C_0402" H 7400 1300 50  0001 C CNN
 F 3 "" H 7400 1300 50  0001 C CNN
 	1    7400 1300
@@
 F 0 "C18" V 7271 1050 50  0000 C CNN
 F 1 "C_Small" V 7362 1050 50  0000 C CNN
-F 2 "Capacitors_SMD:C_0603" H 7500 1050 50  0001 C CNN
+F 2 "Capacitors_SMD:C_0402" H 7500 1050 50  0001 C CNN
 F 3 "" H 7500 1050 50  0001 C CNN
 	1    7500 1050
@@
 F 0 "C12" H 6308 3804 50  0000 R CNN
 F 1 "C_Small" H 6308 3895 50  0000 R CNN
-F 2 "Capacitors_SMD:C_0805" H 6400 3850 50  0001 C CNN
+F 2 "Capacitors_SMD:C_0603" H 6400 3850 50  0001 C CNN
 F 3 "" H 6400 3850 50  0001 C CNN
 	1    6400 3850
@@
 F 0 "C13" H 6558 3804 50  0000 R CNN
 F 1 "C_Small" H 6558 3895 50  0000 R CNN
-F 2 "Capacitors_SMD:C_0603" H 6650 3850 50  0001 C CNN
+F 2 "Capacitors_SMD:C_0402" H 6650 3850 50  0001 C CNN
 F 3 "" H 6650 3850 50  0001 C CNN
 	1    6650 3850
@@
 F 0 "C14" H 6808 4904 50  0000 R CNN
 F 1 "C_Small" H 6808 4995 50  0000 R CNN
-F 2 "Capacitors_SMD:C_0603" H 6900 4950 50  0001 C CNN
+F 2 "Capacitors_SMD:C_0402" H 6900 4950 50  0001 C CNN
 F 3 "" H 6900 4950 50  0001 C CNN
 	1    6900 4950
@@
 F 0 "C19" H 7408 4904 50  0000 R CNN
 F 1 "C_Small" H 7408 4995 50  0000 R CNN
-F 2 "Capacitors_SMD:C_0603" H 7500 4950 50  0001 C CNN
+F 2 "Capacitors_SMD:C_0402" H 7500 4950 50  0001 C CNN
 F 3 "" H 7500 4950 50  0001 C CNN
 	1    7500 4950
@@
 F 0 "C20" H 8008 4904 50  0000 R CNN
 F 1 "C_Small" H 8008 4995 50  0000 R CNN
-F 2 "Capacitors_SMD:C_0603" H 8100 4950 50  0001 C CNN
+F 2 "Capacitors_SMD:C_0402" H 8100 4950 50  0001 C CNN
 F 3 "" H 8100 4950 50  0001 C CNN
 	1    8100 4950
@@
 F 0 "R8" H 6770 4996 50  0000 L CNN
 F 1 "R" H 6770 4905 50  0000 L CNN
-F 2 "Resistors_SMD:R_0603" V 6630 4950 50  0001 C CNN
+F 2 "Resistors_SMD:R_0402" V 6630 4950 50  0001 C CNN
 F 3 "" H 6700 4950 50  0001 C CNN
 	1    6700 4950
@@
 F 0 "R9" H 7420 4996 50  0000 L CNN
 F 1 "R" H 7420 4905 50  0000 L CNN
-F 2 "Resistors_SMD:R_0603" V 7280 4950 50  0001 C CNN
+F 2 "Resistors_SMD:R_0402" V 7280 4950 50  0001 C CNN
 F 3 "" H 7350 4950 50  0001 C CNN
 	1    7350 4950
@@
 F 0 "R11" H 7970 4996 50  0000 L CNN
 F 1 "R" H 7970 4905 50  0000 L CNN
-F 2 "Resistors_SMD:R_0603" V 7830 4950 50  0001 C CNN
+F 2 "Resistors_SMD:R_0402" V 7830 4950 50  0001 C CNN
 F 3 "" H 7900 4950 50  0001 C CNN
 	1    7900 4950
@@
 F 0 "R10" V 7693 1050 50  0000 C CNN
 F 1 "R" V 7784 1050 50  0000 C CNN
-F 2 "Resistors_SMD:R_0603" V 7830 1050 50  0001 C CNN
+F 2 "Resistors_SMD:R_0402" V 7830 1050 50  0001 C CNN
 F 3 "" H 7900 1050 50  0001 C CNN
 	1    7900 1050
@@
 Wire Wire Line
 	9700 4350 9700 4300
+$Sheet
+S 8800 5450 1650 850
+U 5A2E91F4
+F0 "connectors" 60
+F1 "connectors.sch" 60
+$EndSheet
 $EndSCHEMATC

Commit message: Create sub-sheets and start layout
Parts:
- removed C1, C10, C11, C13, C14, C15, C16, C18, C19, C20, C3, C4, C5, C6, C8, C9: C_Small, Capacitors_SMD:C_0402, symbol C_Small
- removed C12, C17, C2, C7: C_Small, Capacitors_SMD:C_0603, symbol C_Small
- removed D1, D2, D3, D4, D5, D6, D7, D8: LED, LEDs:LED_0603, symbol LED
- removed IC1, IC2: ATM90E36_ATM90E36, Housings_QFP:TQFP-48_7x7mm_Pitch0.5mm, symbol ATM90E36_ATM90E36
- removed J1, J2, J3, J4, J5, J6: GS3, Connectors:GS3, symbol GS3
- removed J? (x2): CONN_01X04, Connectors_JST:JST_SH_BM04B-SRSS-TB_04x1.00mm_Straight, symbol CONN_01X04
- removed J? (x2): CONN_01X03, Connectors_JST:JST_SH_BM03B-SRSS-TB_03x1.00mm_Straight, symbol CONN_01X03
- removed R1, R10, R11, R2, R4, R5, R8, R9: R, Resistors_SMD:R_0402, symbol R
- removed R12, R3, R6, R7: SMD-RES-ARRAY, Resistors_SMD:R_Array_Concave_4x0603, symbol SEEED-RESISTOR-2016_SMD-RES-ARRAY-1K-4R_RA1206-8_
- removed Y1, Y2: Crystal_GND24, Crystals:Crystal_SMD_2520-4pin_2.5x2.0mm, symbol Crystal_GND24
Connections:
- net labels removed: +3V3, CF1, CF2, CF3, CF4, CS, DMA, GND, I1N, I1P, I2N, I2P, I3N, I3P, IN, IP, IRQ1, IRQ2, MISO, MOSI, PM0, PM1, SCLK, V1P, V2P, V3P, WARN, ZX0, ZX1, ZX2
- wire segments 278 -> 0
Other:
- note removed: "ATM90E3X Poly Phase Metering AFE"

Commit message: Add manufacturer number and more details on silk
Parts:
- added G1: LOGO, Whatnick_logo:Whatnick_logo, symbol whatnick:LOGO
- added G2: Logo_Open_Hardware_Small, Symbols:OSHW-Logo2_7.3x6mm_SilkScreen, symbol Graphic:Logo_Open_Hardware_Small
- added SYM1: SYM_Flash_Small, Whatnick_logo:Fsilk_HV, symbol Graphic:SYM_Flash_Small
Changed lines of the file:
@@
 F1 "ATM90E36_1.sch" 60
 $EndSheet
+$Comp
+L whatnick:LOGO G1
+U 1 1 5A8F349B
+P 4550 3050
+F 0 "G1" H 4550 2948 60  0001 C CNN
+F 1 "LOGO" H 4550 3152 60  0001 C CNN
+F 2 "Whatnick_logo:Whatnick_logo" H 4550 3050 50  0001 C CNN
+F 3 "" H 4550 3050 50  0001 C CNN
+F 4 " " H 4550 3050 50  0001 C CNN "manf#"
+	1    4550 3050
+	1    0    0    -1
+$EndComp
+$Comp
+L Graphic:Logo_Open_Hardware_Small G2
+U 1 1 5A8F3BBE
+P 5150 3050
+F 0 "G2" H 5150 3325 50  0001 C CNN
+F 1 "Logo_Open_Hardware_Small" H 5150 2825 50  0001 C CNN
+F 2 "Symbols:OSHW-Logo2_7.3x6mm_SilkScreen" H 5150 3050 50  0001 C CNN
+F 3 "~" H 5150 3050 50  0001 C CNN
+F 4 " " H 5150 3050 50  0001 C CNN "manf#"
+	1    5150 3050
+	1    0    0    -1
+$EndComp
+$Comp
+L Graphic:SYM_Flash_Small SYM1
+U 1 1 5A8F3EA0
+P 5750 3050
+F 0 "SYM1" V 5660 3050 50  0001 C CNN
+F 1 "SYM_Flash_Small" V 5840 3050 50  0001 C CNN
+F 2 "Whatnick_logo:Fsilk_HV" H 5750 3025 50  0001 C CNN
+F 3 "~" H 6150 2950 50  0001 C CNN
+F 4 " " H 5750 3050 50  0001 C CNN "manf#"
+	1    5750 3050
+	1    0    0    -1
+$EndComp
 $EndSCHEMATC

Commit message: New BOM output
Parts:
- G1, G2, SYM1: DNP (none) -> (none)
Changed lines of the file:
@@
 F 3 "" H 4550 3050 50  0001 C CNN
 F 4 " " H 4550 3050 50  0001 C CNN "manf#"
+F 5 " " H 4550 3050 50  0001 C CNN "DNP"
 	1    4550 3050
 	1    0    0    -1
@@
 F 3 "~" H 5150 3050 50  0001 C CNN
 F 4 " " H 5150 3050 50  0001 C CNN "manf#"
+F 5 " " H 5150 3050 50  0001 C CNN "DNP"
 	1    5150 3050
 	1    0    0    -1
@@
 F 3 "~" H 6150 2950 50  0001 C CNN
 F 4 " " H 5750 3050 50  0001 C CNN "manf#"
+F 5 " " V 5750 3050 50  0001 C CNN "DNP"
 	1    5750 3050
 	1    0    0    -1
