File: connectors.sch (KiCad schematic (older format))
At the start: 2 parts, among them J7 Conn_01x10, J8 Conn_02x18_Row_Letter_First

Commit message: Create sub-sheets and start layout
Parts:
- J7: footprint (none) -> Molex_board2board:SHDR10W60P200_1X10_2150X400X335P; manf# (none) -> 52418-1010
Changed lines of the file:
@@
 $Descr A4 11693 8268
 encoding utf-8
-Sheet 2 2
+Sheet 2 4
 Title ""
 Date ""
@@
 F 0 "J7" V 3624 1996 50  0000 C CNN
 F 1 "Conn_01x10" V 3715 1996 50  0000 C CNN
-F 2 "" H 3500 2050 50  0001 C CNN
+F 2 "Molex_board2board:SHDR10W60P200_1X10_2150X400X335P" H 3500 2050 50  0001 C CNN
 F 3 "" H 3500 2050 50  0001 C CNN
+F 4 "52418-1010" H 3500 2050 60  0001 C CNN "manf#"
 	1    3500 2050
 	0    1    1    0

Commit message: Add some connector labels
Connections:
- net labels added: 3V3_CPU, 3V3_ISO, CS_0, CS_1, CS_2, GND_CPU, GND_ISO, SCLK, SI/RX, SO/TX
- wire segments 0 -> 25
Changed lines of the file:
@@
 LIBS:ATM90E36_Breakout
 LIBS:din_meter_atm90e36-cache
-EELAYER 26 0
+EELAYER 25 0
 EELAYER END
 $Descr A4 11693 8268
@@
 F 4 "52418-1010" H 3500 2050 60  0001 C CNN "manf#"
 	1    3500 2050
-	0    1    1    0
+	0    -1   -1   0
 $EndComp
 $Comp
@@
 F 3 "" H 6400 1950 50  0001 C CNN
 	1    6400 1950
-	0    1    1    0
+	0    -1   -1   0
 $EndComp
+Text GLabel 3100 2550 3    60   Input ~ 0
+3V3_CPU
+Text GLabel 3200 2550 3    60   Input ~ 0
+GND_CPU
+Text GLabel 3300 2550 3    60   Output ~ 0
+CS_2
+Text GLabel 3400 2550 3    60   Output ~ 0
+CS_0
+Text GLabel 3500 2550 3    60   Output ~ 0
+SCLK
+Text GLabel 3600 2550 3    60   Input ~ 0
+SO/TX
+Text GLabel 3700 2550 3    60   Output ~ 0
+SI/RX
+Text GLabel 3800 2550 3    60   Output ~ 0
+CS_1
+Text GLabel 3900 2550 3    60   BiDi ~ 0
+GND_ISO
+Text GLabel 4000 2550 3    60   BiDi ~ 0
+3V3_ISO
+Text GLabel 5600 2350 3    60   Output ~ 0
+3V3_ISO
+Text GLabel 6300 2350 3    60   Output ~ 0
+GND_ISO
+Wire Wire Line
+	3100 2250 3100 2550
+Wire Wire Line
+	3200 2250 3200 2550
+Wire Wire Line
+	3300 2250 3300 2550
+Wire Wire Line
+	3400 2250 3400 2550
+Wire Wire Line
+	3500 2250 3500 2550
+Wire Wire Line
+	3600 2250 3600 2550
+Wire Wire Line
+	3700 2250 3700 2550
+Wire Wire Line
+	3800 2250 3800 2550
+Wire Wire Line
+	3900 2250 3900 2550
+Wire Wire Line
+	4000 2250 4000 2550
+Wire Wire Line
+	5600 2150 5600 2350
+Wire Wire Line
+	5700 2150 5700 2350
+Wire Wire Line
+	5900 2150 5900 2350
+Wire Wire Line
+	6100 2150 6100 2350
+Wire Wire Line
+	6300 2150 6300 2350
+Wire Wire Line
+	6700 2150 6700 2350
+Wire Wire Line
+	7100 2150 7100 2350
+Wire Wire Line
+	5800 1650 5800 1450
+Wire Wire Line
+	5900 1650 5900 1450
+Wire Wire Line
+	6000 1650 6000 1450
+Wire Wire Line
+	6100 1650 6100 1450
+Wire Wire Line
+	6700 1650 6700 1450
+Wire Wire Line
+	6900 1650 6900 1450
+Wire Wire Line
+	7100 1650 7100 1450
+Wire Wire Line
+	7300 1650 7300 1450
+Text GLabel 6700 2350 3    60   Output ~ 0
+GND_CPU
+Text GLabel 7100 2350 3    60   Output ~ 0
+3V3_CPU
 $EndSCHEMATC

Commit message: Wired up current samplers
Parts:
- added L1, L2: L_Small, Inductors_SMD:L_0402, symbol device:L_Small
- J7: symbol Conn_01x10 -> conn:Conn_01x10
- J8: symbol Conn_02x18_Row_Letter_First -> conn:Conn_02x18_Row_Letter_First
Connections:
- net labels added: +3V3, GND, IA1+, IA1-, IA2+, IA2-, IB1+, IB1-, IB2+, IB2-, IC1+, IC1-, IC2+, IC2-, IN1+, IN1-, IN2+, IN2-, MISO, MOSI, V1P, V2P, V3P
- net labels removed: SI/RX, SO/TX
- wire segments 25 -> 37
Other:
- note added: "Metering to Power/Sampler connector"
Changed lines of the file:
@@
-EESchema Schematic File Version 2
-LIBS:power
-LIBS:device
-LIBS:transistors
-LIBS:conn
-LIBS:linear
-LIBS:regul
-LIBS:74xx
-LIBS:cmos4000
-LIBS:adc-dac
-LIBS:memory
-LIBS:xilinx
-LIBS:microcontrollers
-LIBS:dsp
-LIBS:microchip
-LIBS:analog_switches
-LIBS:motorola
-LIBS:texas
-LIBS:intel
-LIBS:audio
-LIBS:interface
-LIBS:digital-audio
-LIBS:philips
-LIBS:display
-LIBS:cypress
-LIBS:siliconi
-LIBS:opto
-LIBS:atmel
-LIBS:contrib
-LIBS:valves
-LIBS:ATM90E36_Breakout
+EESchema Schematic File Version 4
 LIBS:din_meter_atm90e36-cache
-EELAYER 25 0
+EELAYER 26 0
 EELAYER END
 $Descr A4 11693 8268
@@
 $EndDescr
 $Comp
-L Conn_01x10 J7
+L conn:Conn_01x10 J7
 U 1 1 5A2E938F
 P 3500 2050
@@
 $EndComp
 $Comp
-L Conn_02x18_Row_Letter_First J8
+L conn:Conn_02x18_Row_Letter_First J8
 U 1 1 5A2E95C6
 P 6400 1950
@@
 SCLK
 Text GLabel 3600 2550 3    60   Input ~ 0
-SO/TX
+MISO
 Text GLabel 3700 2550 3    60   Output ~ 0
-SI/RX
+MOSI
 Text GLabel 3800 2550 3    60   Output ~ 0
 CS_1
@@
 Text GLabel 7100 2350 3    60   Output ~ 0
 3V3_CPU
+Text Notes 5600 2950 0    50   ~ 0
+Metering to Power/Sampler connector
+$Comp
+L device:L_Small L1
+U 1 1 5A4B475F
+P 3250 3650
+F 0 "L1" V 3072 3650 50  0000 C CNN
+F 1 "L_Small" V 3163 3650 50  0000 C CNN
+F 2 "Inductors_SMD:L_0402" H 3250 3650 50  0001 C CNN
+F 3 "" H 3250 3650 50  0001 C CNN
+	1    3250 3650
+	0    1    1    0
+$EndComp
+$Comp
+L device:L_Small L2
+U 1 1 5A4B47F5
+P 3250 3900
+F 0 "L2" V 3072 3900 50  0000 C CNN
+F 1 "L_Small" V 3163 3900 50  0000 C CNN
+F 2 "Inductors_SMD:L_0402" H 3250 3900 50  0001 C CNN
+F 3 "" H 3250 3900 50  0001 C CNN
+	1    3250 3900
+	0    1    1    0
+$EndComp
+Wire Wire Line
+	3150 3650 2950 3650
+Wire Wire Line
+	3350 3650 3600 3650
+Wire Wire Line
+	3150 3900 2950 3900
+Wire Wire Line
+	3350 3900 3600 3900
+Text GLabel 2950 3650 0    50   Input ~ 0
+3V3_ISO
+$Comp
+L power:+3V3 #PWR019
+U 1 1 5A4B57CD
+P 3600 3650
+F 0 "#PWR019" H 3600 3500 50  0001 C CNN
+F 1 "+3V3" V 3615 3778 50  0000 L CNN
+F 2 "" H 3600 3650 50  0001 C CNN
+F 3 "" H 3600 3650 50  0001 C CNN
+	1    3600 3650
+	0    1    1    0
+$EndComp
+$Comp
+L power:GND #PWR020
+U 1 1 5A4B583A
+P 3600 3900
+F 0 "#PWR020" H 3600 3650 50  0001 C CNN
+F 1 "GND" V 3605 3772 50  0000 R CNN
+F 2 "" H 3600 3900 50  0001 C CNN
+F 3 "" H 3600 3900 50  0001 C CNN
+	1    3600 3900
+	0    -1   -1   0
+$EndComp
+Text GLabel 2950 3900 0    50   Input ~ 0
+GND_ISO
+Text GLabel 5700 2350 3    50   Output ~ 0
+V1P
+Text GLabel 5900 2350 3    50   Output ~ 0
+V2P
+Text GLabel 6100 2350 3    50   Output ~ 0
+V3P
+Wire Wire Line
+	5600 1650 5600 1450
+Wire Wire Line
+	5700 1650 5700 1450
+Wire Wire Line
+	6200 1650 6200 1450
+Wire Wire Line
+	6300 1650 6300 1450
+Wire Wire Line
+	6400 1650 6400 1450
+Wire Wire Line
+	6500 1650 6500 1450
+Wire Wire Line
+	6800 1650 6800 1450
+Wire Wire Line
+	7000 1650 7000 1450
+Text GLabel 5600 1450 1    50   Output ~ 0
+IA1-
+Text GLabel 5700 1450 1    50   Output ~ 0
+IA1+
+Text GLabel 5800 1450 1    50   Output ~ 0
+IB1-
+Text GLabel 5900 1450 1    50   Output ~ 0
+IB1+
+Text GLabel 6000 1450 1    50   Output ~ 0
+IC1-
+Text GLabel 6100 1450 1    50   Output ~ 0
+IC1+
+Text GLabel 6200 1450 1    50   Output ~ 0
+IC2-
+Text GLabel 6300 1450 1    50   Output ~ 0
+IC2+
+Text GLabel 6400 1450 1    50   Output ~ 0
+IA2-
+Text GLabel 6500 1450 1    50   Output ~ 0
+IA2+
+Text GLabel 6700 1450 1    50   Output ~ 0
+IN1+
+Text GLabel 6900 1450 1    50   Output ~ 0
+IN1-
+Text GLabel 6800 1450 1    50   Output ~ 0
+IB2+
+Text GLabel 7000 1450 1    50   Output ~ 0
+IB2-
+Text GLabel 7100 1450 1    50   Output ~ 0
+IN2+
+Text GLabel 7300 1450 1    50   Output ~ 0
+IN2-
 $EndSCHEMATC

Commit message: New BOM output
Parts:
- J8: DNP (none) -> (none); manf# (none) -> (none)
- L1, L2: manf# (none) -> BLM15BD102SN1D
Changed lines of the file:
@@
 F 2 "Connectors:PCI-EXPRESS" H 6400 1950 50  0001 C CNN
 F 3 "" H 6400 1950 50  0001 C CNN
+F 4 " " H 6400 1950 50  0001 C CNN "manf#"
+F 5 " " V 6400 1950 50  0001 C CNN "DNP"
 	1    6400 1950
 	0    -1   -1   0
@@
 F 2 "Inductors_SMD:L_0402" H 3250 3650 50  0001 C CNN
 F 3 "" H 3250 3650 50  0001 C CNN
+F 4 "BLM15BD102SN1D" H 3250 3650 50  0001 C CNN "manf#"
 	1    3250 3650
 	0    1    1    0
@@
 F 2 "Inductors_SMD:L_0402" H 3250 3900 50  0001 C CNN
 F 3 "" H 3250 3900 50  0001 C CNN
+F 4 "BLM15BD102SN1D" H 3250 3900 50  0001 C CNN "manf#"
 	1    3250 3900
 	0    1    1    0

Commit message: rescue symbols
Parts:
- J7: symbol conn:Conn_01x10 -> din_meter_atm90e36-rescue:Conn_01x10-conn
- J8: symbol conn:Conn_02x18_Row_Letter_First -> din_meter_atm90e36-rescue:Conn_02x18_Row_Letter_First-conn
- L1, L2: symbol device:L_Small -> din_meter_atm90e36-rescue:L_Small-device
Changed lines of the file:
@@
 $EndDescr
 $Comp
-L conn:Conn_01x10 J7
+L din_meter_atm90e36-rescue:Conn_01x10-conn J7
 U 1 1 5A2E938F
 P 3500 2050
@@
 $EndComp
 $Comp
-L conn:Conn_02x18_Row_Letter_First J8
+L din_meter_atm90e36-rescue:Conn_02x18_Row_Letter_First-conn J8
 U 1 1 5A2E95C6
 P 6400 1950
@@
 Metering to Power/Sampler connector
 $Comp
-L device:L_Small L1
+L din_meter_atm90e36-rescue:L_Small-device L1
 U 1 1 5A4B475F
 P 3250 3650
@@
 $EndComp
 $Comp
-L device:L_Small L2
+L din_meter_atm90e36-rescue:L_Small-device L2
 U 1 1 5A4B47F5
 P 3250 3900
